File: PCB/Waveform Generator/Waveform Generator.sch (KiCad schematic (older format))
At the start: 43 parts

Commit message: Working on latest schematic
Parts:
- added C?: 100n, symbol Device:C_Small
- added C? (x4): 15u, symbol Device:C_Small
- added J?: SWD, symbol Connector_Generic:Conn_02x05_Odd_Even
- added J?: USB_B_Micro, symbol Connector:USB_B_Micro
- added J? (x3): Conn_01x02, symbol Connector_Generic:Conn_01x02
- added J? (x2): Conn_01x04, symbol Connector_Generic:Conn_01x04
- added R? (x4): 22, symbol Device:R_Small
- added R? (x8): 1k, symbol Device:R_Small
- added U?: USBLC6-2SC6, Package_TO_SOT_SMD:SOT-23-6, symbol Power_Protection:USBLC6-2SC6
- added U? (x4): OPAMP, symbol pspice:OPAMP
- L?: value L_Small -> 10u
Connections:
- net labels added: ADC1_IN0, ADC1_IN1, DAC_OUT1, DAC_OUT2, SW0, SWCLK, SWDIO, USB_CONN_D+, USB_CONN_D-
- wire segments 88 -> 138
- no-connect marks 1 -> 5
Other:
- note added: "Level Shifting to Signal Output\n"
- note added: "Power"
- note added: "SWD"
- note added: "USB\n"
- moved on the sheet: 12p, 12p?, 16MHz, C?, D?, FB200, R?, SW?

Commit message: PCB Update
Parts:
- added 12p? (x3): 1u, symbol Device:C_Small
- added D?: GREEN, symbol Device:LED_Small
- added D?: RED, symbol Device:LED_Small
- added D?: BLUE, symbol Device:LED_Small
- added J? (x2): Conn_01x04, symbol Connector_Generic:Conn_01x04
- added Q? (x3): Q_NPN_BCE, symbol Device:Q_NPN_BCE
- added R? (x3): 470, symbol Device:R_Small
- added R? (x3): 33, symbol Device:R_Small
- added R? (x2): 2k2, symbol Device:R_Small
- added SW? (x3): Btn1, symbol Switch:SW_Push
Connections:
- net labels added: ADC2_IN0, I2C1_SCL, I2C1_SDA, PB13_Out, PB14_Out, PB15_Out, PC6_Input, PC7_Input, PC8_Input, TIM1_CH1, TIM3_CH1
- net labels removed: ADC1_IN0
- wire segments 138 -> 169
Other:
- note added: "Buttons\n"
- note added: "Connectors\n"
- note added: "LEDs\n"
- moved on the sheet: C?, J?, R?, U?

Commit message: Update
Connections:
- net labels added: USB_ID
- no-connect marks 5 -> 4
Other:
- moved on the sheet: 12p, 12p?, 16MHz, C?, D?, J?, Q?, R?, SW?, U?

Commit message: Working on schematic
Parts:
- added C? (x6): 10n, symbol Device:C_Small
- added PS?: ITP0312D05, symbol Extra~Components:ITP0312D05
- J?: value Conn_01x02 -> 12V Power
- gave numbers to parts that had none: 1
Connections:
- net labels added: -5V, VBUS
- net labels removed: Buck_Out
- wire segments 169 -> 187
Other:
- note added: "12v to +-5v regulator"
- note added: "5v to 3v3\n"
- note removed: "Power"
- note removed: "Step-Down Converter (3v3)\n"
- moved on the sheet: C?, D?, F?, FB?, J?, L?, Q?, R?, SW?

Commit message: Updating schematic
Parts:
- removed D?: RED, symbol Device:LED_Small
- removed R?: 1k, symbol Device:R_Small
- added D?: BLUE, symbol Device:LED_Small
- added H? (x4): MountingHole_Pad, symbol Mechanical:MountingHole_Pad
- added J?: Conn_01x04, symbol Connector_Generic:Conn_01x04
- added Q? (x2): Q_NPN_BCE, symbol Device:Q_NPN_BCE
- added Q?: Q_PNP_BCE, symbol Device:Q_PNP_BCE
- added R? (x4): 1k, symbol Device:R_Small
- added R?: 47, symbol Device:R_Small
- added U?: MAX485E, symbol Interface_UART:MAX485E
Connections:
- net labels added: DE, MAX485_DE, MAX485_PWR, RE, USART1_RX, USART2_RX, USART2_TX
- net labels removed: USART_RX
- wire segments 187 -> 203
Other:
- note added: "Mounting Holes\n"
- note added: "RS485 \n"
- moved on the sheet: 12p, 12p?, 16MHz, C?, D?, F?, FB200, FB?, J?, L?, Q?, R?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

Commit message: Updates
Connections:
- no-connect marks 4 -> 26
Other:
- note added: "Power Circuitry\n"
- moved on the sheet: 12p, 12p?, 16MHz, C?, D?, F?, FB200, FB?, H?, J?, L?, Q?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

Commit message: Making more updates
Parts:
- removed R?: 47k, symbol Device:R_Small
- added D7: GREEN, symbol Device:LED_Small
- added R35: 1k, symbol Device:R_Small
- C11, C12, C13, C24: renamed from 12p?; value 1u -> 12p
- C26: renamed from 12p; value 1u -> 12p
- J2: renamed from J?; value Conn_01x04 -> RS485
- R6: renamed from R?; value 1k5 -> 1k
- gave numbers to parts that had none: 104
- renumbered 16MHz to 16MHz_1, FB200 to FB2
Connections:
- wire segments 203 -> 207
Other:
- moved on the sheet: C1, C10, C2, C3, C4, C5, C6, C7, C8, C9, D1, D2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

Commit message: update
Parts:
- removed J1: 12V Power, symbol Connector_Generic:Conn_01x02
- removed J10, J7, J8, J9: Conn_01x04, symbol Connector_Generic:Conn_01x04
- removed J2: RS485, symbol Connector_Generic:Conn_01x04
- removed J4, J5: Conn_01x02, symbol Connector_Generic:Conn_01x02
- added J1: Power input, symbol Connector:Screw_Terminal_01x02
- added J10: I2C1, symbol Connector:Screw_Terminal_01x04
- added J2: RS485, symbol Connector:Screw_Terminal_01x04
- added J4: Signal 1, symbol Connector:Screw_Terminal_01x02
- added J5: Signal 2, symbol Connector:Screw_Terminal_01x02
- added J7: USART1, symbol Connector:Screw_Terminal_01x04
- added J8: TIMER, symbol Connector:Screw_Terminal_01x04
- added J9: ADC, symbol Connector:Screw_Terminal_01x04
Changed lines of the file:
@@
 DAC_OUT2
-$Comp
-L Connector_Generic:Conn_01x04 J7
-U 1 1 6072C1BC
-P 13900 8500
-F 0 "J7" H 13980 8492 50  0000 L CNN
-F 1 "Conn_01x04" H 13980 8401 50  0000 L CNN
-F 2 "" H 13900 8500 50  0001 C CNN
-F 3 "~" H 13900 8500 50  0001 C CNN
-	1    13900 8500
-	1    0    0    -1
-$EndComp
 $Comp
 L power:GND #PWR0128
@@
 ADC1_IN1
 $Comp
-L Connector_Generic:Conn_01x04 J9
-U 1 1 60730A09
-P 13850 9400
-F 0 "J9" H 13930 9392 50  0000 L CNN
-F 1 "Conn_01x04" H 13930 9301 50  0000 L CNN
-F 2 "" H 13850 9400 50  0001 C CNN
-F 3 "~" H 13850 9400 50  0001 C CNN
-	1    13850 9400
-	1    0    0    -1
-$EndComp
-$Comp
 L power:GND #PWR0130
 U 1 1 60730A0F
@@
 Text GLabel 2900 9650 2    51   Input ~ 0
 I2C1_SCL
-$Comp
-L Connector_Generic:Conn_01x04 J10
-U 1 1 6073F42F
-P 15300 9400
-F 0 "J10" H 15380 9392 50  0000 L CNN
-F 1 "Conn_01x04" H 15380 9301 50  0000 L CNN
-F 2 "" H 15300 9400 50  0001 C CNN
-F 3 "~" H 15300 9400 50  0001 C CNN
-	1    15300 9400
-	1    0    0    -1
-$EndComp
 $Comp
 L power:GND #PWR0132
@@
 Text GLabel 15050 8450 0    51   Input ~ 0
 TIM1_CH1
-$Comp
-L Connector_Generic:Conn_01x04 J8
-U 1 1 60767E94
-P 15250 8450
-F 0 "J8" H 15330 8442 50  0000 L CNN
-F 1 "Conn_01x04" H 15330 8351 50  0000 L CNN
-F 2 "" H 15250 8450 50  0001 C CNN
-F 3 "~" H 15250 8450 50  0001 C CNN
-	1    15250 8450
-	1    0    0    -1
-$EndComp
 $Comp
 L power:GND #PWR0134
@@
 	1    2250 1750
 	1    0    0    1
-$EndComp
-$Comp
-L Connector_Generic:Conn_01x02 J1
-U 1 1 604CA7F0
-P 1150 1750
-F 0 "J1" H 1250 1450 50  0000 C CNN
-F 1 "12V Power" H 1250 1550 50  0000 C CNN
-F 2 "" H 1150 1750 50  0001 C CNN
-F 3 "~" H 1150 1750 50  0001 C CNN
-	1    1150 1750
-	-1   0    0    1
 $EndComp
 $Comp
@@
 	1    0    0    -1
 $EndComp
-$Comp
-L Connector_Generic:Conn_01x04 J2
-U 1 1 60E54529
-P 15250 2450
-F 0 "J2" H 15330 2442 50  0000 L CNN
-F 1 "RS485" H 15330 2351 50  0000 L CNN
-F 2 "" H 15250 2450 50  0001 C CNN
-F 3 "~" H 15250 2450 50  0001 C CNN
-	1    15250 2450
-	1    0    0    -1
-$EndComp
 Text GLabel 13850 2350 0    50   Input ~ 0
 USART2_RX
@@
 $EndComp
 $Comp
-L Connector_Generic:Conn_01x02 J5
-U 1 1 605B4C62
-P 9550 8950
-F 0 "J5" H 9630 8942 50  0000 L CNN
-F 1 "Conn_01x02" H 9630 8851 50  0000 L CNN
-F 2 "" H 9550 8950 50  0001 C CNN
-F 3 "~" H 9550 8950 50  0001 C CNN
-	1    9550 8950
-	1    0    0    -1
-$EndComp
-$Comp
-L Connector_Generic:Conn_01x02 J4
-U 1 1 605A009D
-P 9550 7500
-F 0 "J4" H 9630 7492 50  0000 L CNN
-F 1 "Conn_01x02" H 9630 7401 50  0000 L CNN
-F 2 "" H 9550 7500 50  0001 C CNN
-F 3 "~" H 9550 7500 50  0001 C CNN
-	1    9550 7500
-	1    0    0    -1
-$EndComp
-$Comp
 L power:GND #PWR0170
 U 1 1 605A00A9
@@
 	4500 9300 4500 9350
 Connection ~ 4500 9350
-Connection ~ 1350 1650
 Wire Wire Line
 	2000 7150 2100 7150
@@
 Wire Notes Line
 	700  750  10800 750
+$Comp
+L Connector:Screw_Terminal_01x02 J1
+U 1 1 61627931
+P 1150 1750
+F 0 "J1" H 1200 1450 50  0000 C CNN
+F 1 "Power input" H 1250 1550 50  0000 C CNN
+F 2 "" H 1150 1750 50  0001 C CNN
+F 3 "~" H 1150 1750 50  0001 C CNN
+	1    1150 1750
+	-1   0    0    1
+$EndComp
+Connection ~ 1350 1650
+$Comp
+L Connector:Screw_Terminal_01x04 J2
+U 1 1 61629C36
+P 15250 2450
+F 0 "J2" H 15330 2442 50  0000 L CNN
+F 1 "RS485" H 15330 2351 50  0000 L CNN
+F 2 "" H 15250 2450 50  0001 C CNN
+F 3 "~" H 15250 2450 50  0001 C CNN
+	1    15250 2450
+	1    0    0    -1
+$EndComp
+$Comp
+L Connector:Screw_Terminal_01x02 J4
+U 1 1 6162CC34
+P 9550 7500
+F 0 "J4" H 9630 7492 50  0000 L CNN
+F 1 "Signal 1" H 9630 7401 50  0000 L CNN
+F 2 "" H 9550 7500 50  0001 C CNN
+F 3 "~" H 9550 7500 50  0001 C CNN
+	1    9550 7500
+	1    0    0    -1
+$EndComp
+$Comp
+L Connector:Screw_Terminal_01x02 J5
+U 1 1 6162DCDE
+P 9550 8950
+F 0 "J5" H 9630 8942 50  0000 L CNN
+F 1 "Signal 2" H 9630 8851 50  0000 L CNN
+F 2 "" H 9550 8950 50  0001 C CNN
+F 3 "~" H 9550 8950 50  0001 C CNN
+	1    9550 8950
+	1    0    0    -1
+$EndComp
+$Comp
+L Connector:Screw_Terminal_01x04 J7
+U 1 1 6162F55F
+P 13900 8500
+F 0 "J7" H 13980 8492 50  0000 L CNN
+F 1 "USART1" H 13980 8401 50  0000 L CNN
+F 2 "" H 13900 8500 50  0001 C CNN
+F 3 "~" H 13900 8500 50  0001 C CNN
+	1    13900 8500
+	1    0    0    -1
+$EndComp
+$Comp
+L Connector:Screw_Terminal_01x04 J10
+U 1 1 61630A48
+P 15300 9400
+F 0 "J10" H 15380 9392 50  0000 L CNN
+F 1 "I2C1" H 15380 9301 50  0000 L CNN
+F 2 "" H 15300 9400 50  0001 C CNN
+F 3 "~" H 15300 9400 50  0001 C CNN
+	1    15300 9400
+	1    0    0    -1
+$EndComp
+$Comp
+L Connector:Screw_Terminal_01x04 J8
+U 1 1 616310F5
+P 15250 8450
+F 0 "J8" H 15330 8442 50  0000 L CNN
+F 1 "TIMER" H 15330 8351 50  0000 L CNN
+F 2 "" H 15250 8450 50  0001 C CNN
+F 3 "~" H 15250 8450 50  0001 C CNN
+	1    15250 8450
+	1    0    0    -1
+$EndComp
+$Comp
+L Connector:Screw_Terminal_01x04 J9
+U 1 1 6163141B
+P 13850 9400
+F 0 "J9" H 13930 9392 50  0000 L CNN
+F 1 "ADC" H 13930 9301 50  0000 L CNN
+F 2 "" H 13850 9400 50  0001 C CNN
+F 3 "~" H 13850 9400 50  0001 C CNN
+	1    13850 9400
+	1    0    0    -1
+$EndComp
 $EndSCHEMATC
