File: PCB/Waveform Generator/Waveform Generator.sch (KiCad schematic (older format))
At the start: 115 parts, among them J1 Power input, J10 I2C1, J2 RS485, J3 USB_B_Micro, J4 Signal 1, J5 Signal 2, J6 SWD, J7 USART1, J8 TIMER, J9 ADC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

Commit message: Schematic mostly done
Parts:
- added U8: LM335ADT, symbol Extra~Components:LM335ADT
- renumbered D7 to D8
Connections:
- net labels added: TEMP_SENSE
- no-connect marks 26 -> 25
Other:
- note added: "TEMP SENSE\n"
- moved on the sheet: C11, C12, C13, SW4, SW5, SW6

Commit message: Working on schematic footprints
Parts:
- added J11, J12, J13, J14, J15, J16, J17, J18: 5001, symbol Extra~Components:5001
- C1, C2: footprint (none) -> Capacitor_SMD:C_1206_3216Metric
- C10, C3, C4, C5, C6, C7, C8, C9: footprint (none) -> Capacitor_SMD:C_0603_1608Metric
- C11, C12, C13, C14, C15, C16, C17, C18, C19, C20, C21, C24, C25, C26, C27, C28, C29, C30, C31: footprint (none) -> Capacitor_SMD:C_0402_1005Metric
- C22, C23: value 100n -> 2.2u; footprint (none) -> Capacitor_SMD:C_0603_1608Metric
- D1, D2: footprint (none) -> Diode_SMD:D_SOD-123
- D3, D4, D5, D6, D7, D8: footprint (none) -> LED_SMD:LED_0603_1608Metric
- F1: footprint (none) -> Fuse:Fuse_1206_3216Metric
- FB1, FB2: footprint (none) -> Inductor_SMD:L_1206_3216Metric
- H1, H2, H3, H4: footprint (none) -> MountingHole:MountingHole_4.3mm_M4_Pad_Via
- J1, J4, J5: footprint (none) -> TerminalBlock_MetzConnect:TerminalBlock_MetzConnect_Type086_RT03402HBLC_1x02_P3.81mm_Horizontal
- J10, J2, J7, J8, J9: footprint (none) -> TerminalBlock_MetzConnect:TerminalBlock_MetzConnect_Type086_RT03404HBLC_1x04_P3.81mm_Horizontal
- J3: footprint (none) -> Connector_USB:USB_Micro-B_Molex-105017-0001
- J6: footprint (none) -> Connector_PinSocket_1.27mm:PinSocket_2x05_P1.27mm_Vertical
Connections:
- net labels added: BT3N_Input, BTN1_Input, BTN2_Input, BTN3_Input, LED1, LED2, LED3
- net labels removed: PB13_Out, PB14_Out, PB15_Out, PC6_Input, PC7_Input, PC8_Input
- wire segments 207 -> 221
Other:
- moved on the sheet: C11, C12, C13, H1, H2, H3, H4, SW4, SW5, SW6

Commit message: Almost done with component footprints
Parts:
- J11, J12, J13, J14, J15, J16, J17, J18: footprint (none) -> Extra Components:5001 Test Point
- L1: footprint (none) -> Inductor_SMD:L_Sunlord_MWSA0518_5.4x5.2mm
- PS1: footprint (none) -> Extra Components:ITP0312D05
- PS2: footprint (none) -> Package_TO_SOT_SMD:SOT-23-6
- Q1, Q2, Q3, Q4, Q5, Q6: footprint (none) -> Package_TO_SOT_SMD:SOT-23
- R1, R10, R2, R24, R26, R28, R3, R35, R4, R5, R6, R8, R9: footprint (none) -> Resistor_SMD:R_0603_1608Metric
- R11, R12, R13, R14, R15, R16, R17, R18, R19, R20, R21, R22, R23, R25, R27, R29, R30, R31, R32, R33, R34, R7: footprint (none) -> Resistor_SMD:R_0402_1005Metric
- SW1, SW3: footprint (none) -> Button_Switch_SMD:SW_SPDT_PCM12
- SW2, SW4, SW5, SW6: footprint (none) -> Extra Components:TS-1109S-B-B
- U2, U8: footprint (none) -> Package_SO:SOIC-8-1EP_3.9x4.9mm_P1.27mm_EP2.29x3mm
- U4, U5, U6, U7: footprint (none) -> Package_SO:MSOP-8-1EP_3x3mm_P0.65mm_EP1.68x1.88mm

Commit message: Working on schematic
Parts:
- 16MHz_1: footprint (none) -> Crystal:Crystal_SMD_3225-4Pin_3.2x2.5mm
Changed lines of the file:
@@
 F 0 "16MHz_1" H 4000 9550 50  0000 L CNN
 F 1 "Y200" H 4050 9650 50  0000 L CNN
-F 2 "" H 4150 9350 50  0001 C CNN
+F 2 "Crystal:Crystal_SMD_3225-4Pin_3.2x2.5mm" H 4150 9350 50  0001 C CNN
 F 3 "~" H 4150 9350 50  0001 C CNN
 	1    4150 9350

Commit message: Starting PCB layout
Parts:
- removed J12: 5001, Extra Components:5001 Test Point, symbol Extra~Components:5001
- removed J4: Signal 1, TerminalBlock_MetzConnect:TerminalBlock_MetzConnect_Type086_RT03402HBLC_1x02_P3.81mm_Horizontal, symbol Connector:Screw_Terminal_01x02
- removed U4, U5, U6, U7: OPAMP, Package_SO:MSOP-8-1EP_3x3mm_P0.65mm_EP1.68x1.88mm, symbol pspice:OPAMP
- added J12: Signal 2, TerminalBlock_MetzConnect:TerminalBlock_MetzConnect_Type086_RT03402HBLC_1x02_P3.81mm_Horizontal, symbol Connector:Screw_Terminal_01x02
- added J4: 5001, Extra Components:5001 Test Point, symbol Extra~Components:5001
- added U4, U5: LTC2051HVIMS8, Package_SO:MSOP-8-1EP_3x3mm_P0.65mm_EP1.73x1.85mm, symbol Extra~Components:LTC2051HVIMS8
Connections:
- wire segments 221 -> 217
Other:
- moved on the sheet: C30, R21

Commit message: Working
Parts:
- added D8: GREEN, LED_SMD:LED_0603_1608Metric, symbol Device:LED_Small
- added R35: 1k, Resistor_SMD:R_0603_1608Metric, symbol Device:R_Small
- PS1: value ITP0312D05 -> ITP0324D05
Changed lines of the file:
@@
 	8750 1700 8750 1600
-$Comp
-L Device:R_Small R6
-U 1 1 60360DB4
-P 9550 2000
-F 0 "R6" H 9609 2046 50  0000 L CNN
-F 1 "1k" H 9609 1955 50  0000 L CNN
-F 2 "Resistor_SMD:R_0603_1608Metric" H 9550 2000 50  0001 C CNN
-F 3 "~" H 9550 2000 50  0001 C CNN
-	1    9550 2000
-	1    0    0    -1
-$EndComp
-$Comp
-L power:GND #PWR0127
-U 1 1 60361815
-P 9550 2100
-F 0 "#PWR0127" H 9550 1850 50  0001 C CNN
-F 1 "GND" H 9555 1927 50  0000 C CNN
-F 2 "" H 9550 2100 50  0001 C CNN
-F 3 "" H 9550 2100 50  0001 C CNN
-	1    9550 2100
-	1    0    0    -1
-$EndComp
 $Comp
 L Switch:SW_SPDT SW1
@@
 $EndComp
 NoConn ~ 10150 1700
-Wire Wire Line
-	9550 1600 9550 1700
-$Comp
-L Device:LED_Small D3
-U 1 1 6035F732
-P 9550 1800
-F 0 "D3" V 9596 1732 50  0000 R CNN
-F 1 "GREEN" V 9505 1732 50  0000 R CNN
-F 2 "LED_SMD:LED_0603_1608Metric" V 9550 1800 50  0001 C CNN
-F 3 "~" V 9550 1800 50  0001 C CNN
-	1    9550 1800
-	0    -1   -1   0
-$EndComp
 Text Notes 5600 1250 0    47   ~ 0
 5v to 3v3\n
 Connection ~ 8750 1600
-Wire Wire Line
-	9550 1600 9750 1600
-Connection ~ 9550 1600
 Text Notes 9350 1250 0    47   ~ 0
 Pwr LED and Switch
@@
 P 2900 1800
 F 0 "PS1" H 2900 2200 59  0000 C CNN
-F 1 "ITP0312D05" H 2900 2100 59  0000 C CNN
+F 1 "ITP0324D05" H 2900 2100 59  0000 C CNN
 F 2 "Extra Components:ITP0312D05" H 3100 1800 59  0001 C CNN
 F 3 "" H 3100 1800 59  0001 C CNN
@@
 	8850 1600 8850 1500
 Connection ~ 8850 1600
-Wire Wire Line
-	8850 1600 9550 1600
 $Comp
 L Extra~Components:5001 J17
@@
 Wire Notes Line
 	6400 9250 6400 6400
+Wire Wire Line
+	8850 1600 9550 1600
+Wire Wire Line
+	9550 1600 9750 1600
+Connection ~ 9550 1600
+Wire Wire Line
+	9550 1600 9550 1700
+$Comp
+L Device:LED_Small D3
+U 1 1 6035F732
+P 9550 1800
+F 0 "D3" V 9596 1732 50  0000 R CNN
+F 1 "GREEN" V 9505 1732 50  0000 R CNN
+F 2 "LED_SMD:LED_0603_1608Metric" V 9550 1800 50  0001 C CNN
+F 3 "~" V 9550 1800 50  0001 C CNN
+	1    9550 1800
+	0    -1   -1   0
+$EndComp
+$Comp
+L power:GND #PWR0127
+U 1 1 60361815
+P 9550 2100
+F 0 "#PWR0127" H 9550 1850 50  0001 C CNN
+F 1 "GND" H 9555 1927 50  0000 C CNN
+F 2 "" H 9550 2100 50  0001 C CNN
+F 3 "" H 9550 2100 50  0001 C CNN
+	1    9550 2100
+	1    0    0    -1
+$EndComp
+$Comp
+L Device:R_Small R6
+U 1 1 60360DB4
+P 9550 2000
+F 0 "R6" H 9609 2046 50  0000 L CNN
+F 1 "1k" H 9609 1955 50  0000 L CNN
+F 2 "Resistor_SMD:R_0603_1608Metric" H 9550 2000 50  0001 C CNN
+F 3 "~" H 9550 2000 50  0001 C CNN
+	1    9550 2000
+	1    0    0    -1
+$EndComp
+$Comp
+L Device:LED_Small D8
+U 1 1 6031020B
+P 4350 1700
+F 0 "D8" V 4396 1632 50  0000 R CNN
+F 1 "GREEN" V 4305 1632 50  0000 R CNN
+F 2 "LED_SMD:LED_0603_1608Metric" V 4350 1700 50  0001 C CNN
+F 3 "~" V 4350 1700 50  0001 C CNN
+	1    4350 1700
+	0    -1   -1   0
+$EndComp
+$Comp
+L power:GND #PWR?
+U 1 1 60310211
+P 4350 2000
+F 0 "#PWR?" H 4350 1750 50  0001 C CNN
+F 1 "GND" H 4355 1827 50  0000 C CNN
+F 2 "" H 4350 2000 50  0001 C CNN
+F 3 "" H 4350 2000 50  0001 C CNN
+	1    4350 2000
+	1    0    0    -1
+$EndComp
+$Comp
+L Device:R_Small R35
+U 1 1 60310217
+P 4350 1900
+F 0 "R35" H 4409 1946 50  0000 L CNN
+F 1 "1k" H 4409 1855 50  0000 L CNN
+F 2 "Resistor_SMD:R_0603_1608Metric" H 4350 1900 50  0001 C CNN
+F 3 "~" H 4350 1900 50  0001 C CNN
+	1    4350 1900
+	1    0    0    -1
+$EndComp
 $EndSCHEMATC

Commit message: New OP-amps and regulators
Parts:
- removed C29, C30: 15u, Capacitor_SMD:C_0402_1005Metric, symbol Device:C_Small
- removed D2: B5819W, Diode_SMD:D_SOD-123, symbol Device:D_Schottky_Small
- removed J11: 5001, Extra Components:5001 Test Point, symbol Extra~Components:5001
- removed J12: Signal 2, TerminalBlock_MetzConnect:TerminalBlock_MetzConnect_Type086_RT03402HBLC_1x02_P3.81mm_Horizontal, symbol Connector:Screw_Terminal_01x02
- removed L1: 10u, Inductor_SMD:L_Sunlord_MWSA0518_5.4x5.2mm, symbol Device:L_Small
- removed PS2: MP2359DJ-LF-Z, Package_TO_SOT_SMD:SOT-23-6, symbol Extra~Components:MP2359DJ-LF-Z
- removed R1: 100k, Resistor_SMD:R_0603_1608Metric, symbol Device:R_Small
- removed R19, R20, R21, R22: 1k, Resistor_SMD:R_0402_1005Metric, symbol Device:R_Small
- removed R2: 68k, Resistor_SMD:R_0603_1608Metric, symbol Device:R_Small
- removed R3: 47k, Resistor_SMD:R_0603_1608Metric, symbol Device:R_Small
- removed R4: 15k, Resistor_SMD:R_0603_1608Metric, symbol Device:R_Small
- removed R5: 270, Resistor_SMD:R_0603_1608Metric, symbol Device:R_Small
- removed U4, U5: LTC2051HVIMS8, Package_SO:MSOP-8-1EP_3x3mm_P0.65mm_EP1.73x1.85mm, symbol Extra~Components:LTC2051HVIMS8
- added C? (x2): 15u, Capacitor_SMD:C_0402_1005Metric, symbol Device:C_Small
- added J?: Signal 2, TerminalBlock_MetzConnect:TerminalBlock_MetzConnect_Type086_RT03402HBLC_1x02_P3.81mm_Horizontal, symbol Connector:Screw_Terminal_01x02
- added J?: 5001, Extra Components:5001 Test Point, symbol Extra~Components:5001
- added PS2: AMS1117-3.3, Package_TO_SOT_SMD:SOT-223-3_TabPin2, symbol Regulator_Linear:AMS1117-3.3
- added R? (x4): 1k, Resistor_SMD:R_0402_1005Metric, symbol Device:R_Small
- added U4, U? (x3): OPA1602, symbol Amplifier_Operational:OPA1602
- added U6: STM32F439ZITx, Package_QFP:LQFP-144_20x20mm_P0.5mm, symbol MCU_ST_STM32F4:STM32F439ZITx
- C8: value 10n -> 0.1u
- C9: value 10u -> 0.1u
- renumbered D8 to D9, R35 to R36
Connections:
- wire segments 217 -> 192
Other:
- moved on the sheet: C27, C28, D3, D8, J5, R15, R16, R17, R18, R35, R6, SW1

Commit message: Updating op-amps and powersupply
Parts:
- removed U6: STM32F439ZITx, Package_QFP:LQFP-144_20x20mm_P0.5mm, symbol MCU_ST_STM32F4:STM32F439ZITx
- U4: footprint (none) -> Package_SO:SOP-8_3.9x4.9mm_P1.27mm
- U5: renamed from U?; footprint (none) -> Package_SO:SOP-8_3.9x4.9mm_P1.27mm
- gave numbers to parts that had none: 8
Changed lines of the file:
@@
-$EndComp
-$Comp
-L MCU_ST_STM32F4:STM32F439ZITx U6
-U 1 1 6031F6E7
-P -1500 8750
-F 0 "U6" H -1500 5061 50  0000 C CNN
-F 1 "STM32F439ZITx" H -1500 4970 50  0000 C CNN
-F 2 "Package_QFP:LQFP-144_20x20mm_P0.5mm" H -2500 5350 50  0001 R CNN
-F 3 "http://www.st.com/st-web-ui/static/active/en/resource/technical/document/datasheet/DM00077036.pdf" H -1500 8750 50  0001 C CNN
-	1    -1500 8750
-	1    0    0    -1
 $EndComp
 $Comp
@@
 F 0 "U4" H 7650 7717 50  0000 C CNN
 F 1 "OPA1602" H 7650 7626 50  0000 C CNN
-F 2 "" H 7650 7350 50  0001 C CNN
+F 2 "Package_SO:SOP-8_3.9x4.9mm_P1.27mm" H 7650 7350 50  0001 C CNN
 F 3 "http://www.ti.com/lit/ds/symlink/opa1604.pdf" H 7650 7350 50  0001 C CNN
 	1    7650 7350
@@
 F 0 "U4" H 8650 7617 50  0000 C CNN
 F 1 "OPA1602" H 8650 7526 50  0000 C CNN
-F 2 "" H 8650 7250 50  0001 C CNN
+F 2 "Package_SO:SOP-8_3.9x4.9mm_P1.27mm" H 8650 7250 50  0001 C CNN
 F 3 "http://www.ti.com/lit/ds/symlink/opa1604.pdf" H 8650 7250 50  0001 C CNN
 	2    8650 7250
@@
 F 0 "U4" H 9908 7346 50  0000 L CNN
 F 1 "OPA1602" H 9908 7255 50  0000 L CNN
-F 2 "" H 9950 7300 50  0001 C CNN
+F 2 "Package_SO:SOP-8_3.9x4.9mm_P1.27mm" H 9950 7300 50  0001 C CNN
 F 3 "http://www.ti.com/lit/ds/symlink/opa1604.pdf" H 9950 7300 50  0001 C CNN
 	3    9950 7300
@@
 	9150 7250 8950 7250
 $Comp
-L Connector:Screw_Terminal_01x02 J?
+L Connector:Screw_Terminal_01x02 J12
 U 1 1 607192B2
 P 9350 8350
-F 0 "J?" H 9430 8342 50  0000 L CNN
+F 0 "J12" H 9430 8342 50  0000 L CNN
 F 1 "Signal 2" H 9430 8251 50  0000 L CNN
 F 2 "TerminalBlock_MetzConnect:TerminalBlock_MetzConnect_Type086_RT03402HBLC_1x02_P3.81mm_Horizontal" H 9350 8350 50  0001 C CNN
@@
 $EndComp
 $Comp
-L power:GND #PWR?
+L power:GND #PWR010
 U 1 1 607192B8
 P 9150 8450
-F 0 "#PWR?" H 9150 8200 50  0001 C CNN
+F 0 "#PWR010" H 9150 8200 50  0001 C CNN
 F 1 "GND" H 9155 8277 50  0000 C CNN
 F 2 "" H 9150 8450 50  0001 C CNN
@@
 $EndComp
 $Comp
-L Device:R_Small R?
+L Device:R_Small R3
 U 1 1 607192BE
 P 8750 8600
-F 0 "R?" V 8850 8600 50  0000 C CNN
+F 0 "R3" V 8850 8600 50  0000 C CNN
 F 1 "1k" V 8750 8600 50  0000 C CNN
 F 2 "Resistor_SMD:R_0402_1005Metric" H 8750 8600 50  0001 C CNN
@@
 $EndComp
 $Comp
-L power:GND #PWR?
+L power:GND #PWR08
 U 1 1 607192C4
 P 8350 8250
-F 0 "#PWR?" H 8350 8000 50  0001 C CNN
+F 0 "#PWR08" H 8350 8000 50  0001 C CNN
 F 1 "GND" V 8400 8100 50  0000 C CNN
 F 2 "" H 8350 8250 50  0001 C CNN
@@
 	8650 8600 8350 8600
 $Comp
-L power:+5V #PWR?
+L power:+5V #PWR07
 U 1 1 607192CB
 P 9850 8100
-F 0 "#PWR?" H 9850 7950 50  0001 C CNN
+F 0 "#PWR07" H 9850 7950 50  0001 C CNN
 F 1 "+5V" H 9865 8273 50  0000 C CNN
 F 2 "" H 9850 8100 50  0001 C CNN
@@
 $EndComp
 $Comp
-L Device:R_Small R?
+L Device:R_Small R4
 U 1 1 607192D1
 P 7550 8750
-F 0 "R?" H 7450 8850 50  0000 C CNN
+F 0 "R4" H 7450 8850 50  0000 C CNN
 F 1 "1k" H 7450 8800 50  0000 C CNN
 F 2 "Resistor_SMD:R_0402_1005Metric" H 7550 8750 50  0001 C CNN
@@
 $EndComp
 $Comp
-L power:GND #PWR?
+L power:GND #PWR09
 U 1 1 607192D7
 P 7350 8350
-F 0 "#PWR?" H 7350 8100 50  0001 C CNN
+F 0 "#PWR09" H 7350 8100 50  0001 C CNN
 F 1 "GND" V 7400 8200 50  0000 C CNN
 F 2 "" H 7350 8350 50  0001 C CNN
@@
 $EndComp
 $Comp
-L Device:R_Small R?
+L Device:R_Small R1
 U 1 1 607192DD
 P 8050 8450
-F 0 "R?" V 8150 8450 50  0000 C CNN
+F 0 "R1" V 8150 8450 50  0000 C CNN
 F 1 "1k" V 7945 8450 50  0000 C CNN
 F 2 "Resistor_SMD:R_0402_1005Metric" H 8050 8450 50  0001 C CNN
@@
 $EndComp
 $Comp
-L Device:C_Small C?
+L Device:C_Small C29
 U 1 1 607192E3
 P 8250 8450
-F 0 "C?" V 8200 8250 50  0000 L CNN
+F 0 "C29" V 8200 8250 50  0000 L CNN
 F 1 "15u" V 8300 8250 50  0000 L CNN
 F 2 "Capacitor_SMD:C_0402_1005Metric" H 8250 8450 50  0001 C CNN
@@
 $EndComp
 $Comp
-L Amplifier_Operational:OPA1602 U?
+L Amplifier_Operational:OPA1602 U5
 U 1 1 607192E9
 P 7650 8450
-F 0 "U?" H 7650 8817 50  0000 C CNN
+F 0 "U5" H 7650 8817 50  0000 C CNN
 F 1 "OPA1602" H 7650 8726 50  0000 C CNN
-F 2 "" H 7650 8450 50  0001 C CNN
+F 2 "Package_SO:SOP-8_3.9x4.9mm_P1.27mm" H 7650 8450 50  0001 C CNN
 F 3 "http://www.ti.com/lit/ds/symlink/opa1604.pdf" H 7650 8450 50  0001 C CNN
 	1    7650 8450
@@
 $EndComp
 $Comp
-L Amplifier_Operational:OPA1602 U?
+L Amplifier_Operational:OPA1602 U5
 U 2 1 607192EF
 P 8650 8350
-F 0 "U?" H 8650 8717 50  0000 C CNN
+F 0 "U5" H 8650 8717 50  0000 C CNN
 F 1 "OPA1602" H 8650 8626 50  0000 C CNN
-F 2 "" H 8650 8350 50  0001 C CNN
+F 2 "Package_SO:SOP-8_3.9x4.9mm_P1.27mm" H 8650 8350 50  0001 C CNN
 F 3 "http://www.ti.com/lit/ds/symlink/opa1604.pdf" H 8650 8350 50  0001 C CNN
 	2    8650 8350
@@
 $EndComp
 $Comp
-L Amplifier_Operational:OPA1602 U?
+L Amplifier_Operational:OPA1602 U5
 U 3 1 607192F5
 P 9950 8400
-F 0 "U?" H 9908 8446 50  0000 L CNN
+F 0 "U5" H 9908 8446 50  0000 L CNN
 F 1 "OPA1602" H 9908 8355 50  0000 L CNN
-F 2 "" H 9950 8400 50  0001 C CNN
+F 2 "Package_SO:SOP-8_3.9x4.9mm_P1.27mm" H 9950 8400 50  0001 C CNN
 F 3 "http://www.ti.com/lit/ds/symlink/opa1604.pdf" H 9950 8400 50  0001 C CNN
 	3    9950 8400
@@
 $EndComp
 $Comp
-L Device:C_Small C?
+L Device:C_Small C30
 U 1 1 607192FB
 P 7250 8550
-F 0 "C?" V 7200 8600 50  0000 L CNN
+F 0 "C30" V 7200 8600 50  0000 L CNN
 F 1 "15u" V 7350 8550 50  0000 L CNN
 F 2 "Capacitor_SMD:C_0402_1005Metric" H 7250 8550 50  0001 C CNN
@@
 $EndComp
 $Comp
-L Device:R_Small R?
+L Device:R_Small R2
 U 1 1 60719301
 P 7000 8550
-F 0 "R?" V 6804 8550 50  0000 C CNN
+F 0 "R2" V 6804 8550 50  0000 C CNN
 F 1 "1k" V 6895 8550 50  0000 C CNN
 F 2 "Resistor_SMD:R_0402_1005Metric" H 7000 8550 50  0001 C CNN
@@
 	7950 8750 7950 8450
 $Comp
-L power:-5V #PWR?
+L power:-5V #PWR011
 U 1 1 6071930D
 P 9850 8700
-F 0 "#PWR?" H 9850 8800 50  0001 C CNN
+F 0 "#PWR011" H 9850 8800 50  0001 C CNN
 F 1 "-5V" V 9800 8900 50  0000 C CNN
 F 2 "" H 9850 8700 50  0001 C CNN
@@
 	8950 8600 8950 8350
 $Comp
-L Extra~Components:5001 J?
+L Extra~Components:5001 J11
 U 1 1 60719318
 P 8950 8200
-F 0 "J?" V 9150 8150 59  0000 L CNN
+F 0 "J11" V 9150 8150 59  0000 L CNN
 F 1 "5001" V 9050 8100 59  0000 L CNN
 F 2 "Extra Components:5001 Test Point" H 9000 8150 59  0001 C CNN
