File: PCB/Waveform Generator/Waveform Generator.sch (KiCad schematic (older format))
At the start: 117 parts, among them J1 Power input, J10 I2C1, J11 5001, J12 Signal 2, J13 5001, J14 5001, J15 5001, J16 5001, J17 5001, J18 5001, J2 RS485, J3 USB_B_Micro, J4 5001, J5 Signal 2, J6 SWD, J7 USART1, J8 TIMER, J9 ADC, Q0 AO3401A, Q1 Q_NPN_BCE, Q2 Q_NPN_BCE, Q3 Q_PNP_BCE, Q4 Q_NPN_BCE, Q5 Q_NPN_BCE, Q6 Q_NPN_BCE, SW1 SW_SPDT, SW2 RESET Button, SW3 SW_SPDT, SW4 Btn1, SW5 Btn1, SW6 Btn1, U1 STM32F405RGT6, U2 MAX485E, U3 USBLC6-2SC6, U4 OPA1602, U5 OPA1602, U8 LM335ADT

Commit message: Making updates to schematic
Parts:
- added U10, U11, U6, U7, U9: USBLC6-2SC6, Package_TO_SOT_SMD:SOT-23-6, symbol Power_Protection:USBLC6-2SC6
Connections:
- wire segments 192 -> 212
Other:
- moved on the sheet: 16MHz_1, C11, C12, C13, C14, C15, C16, C17, C18, C19, C20, C21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

Commit message: Working on next chip
Parts:
- added C? (x2): 2.2u, Capacitor_SMD:C_0603_1608Metric, symbol Device:C_Small
- added U?: STM32F429ZITx, Package_QFP:LQFP-144_20x20mm_P0.5mm, symbol MCU_ST_STM32F4:STM32F429ZITx
Connections:
- wire segments 212 -> 236
Changed lines of the file:
@@
 Wire Notes Line
 	11450 9900 16000 9900
+$Comp
+L MCU_ST_STM32F4:STM32F429ZITx U?
+U 1 1 60B20EB9
+P -4600 9700
+F 0 "U?" H -3850 6150 50  0000 C CNN
+F 1 "STM32F429ZITx" H -3800 6000 50  0000 C CNN
+F 2 "Package_QFP:LQFP-144_20x20mm_P0.5mm" H -5600 6300 50  0001 R CNN
+F 3 "http://www.st.com/st-web-ui/static/active/en/resource/technical/document/datasheet/DM00071990.pdf" H -4600 9700 50  0001 C CNN
+	1    -4600 9700
+	1    0    0    -1
+$EndComp
+Wire Wire Line
+	-5200 6100 -5100 6100
+Connection ~ -5100 6100
+Wire Wire Line
+	-5100 6100 -5000 6100
+Connection ~ -5000 6100
+Wire Wire Line
+	-5000 6100 -4900 6100
+Connection ~ -4900 6100
+Wire Wire Line
+	-4900 6100 -4800 6100
+Connection ~ -4800 6100
+Wire Wire Line
+	-4800 6100 -4700 6100
+Connection ~ -4700 6100
+Wire Wire Line
+	-4700 6100 -4600 6100
+Connection ~ -4600 6100
+Wire Wire Line
+	-4600 6100 -4500 6100
+Connection ~ -4500 6100
+Wire Wire Line
+	-4500 6100 -4400 6100
+Connection ~ -4400 6100
+Wire Wire Line
+	-4400 6100 -4300 6100
+Connection ~ -4300 6100
+Wire Wire Line
+	-4300 6100 -4200 6100
+Connection ~ -4200 6100
+Wire Wire Line
+	-4200 6100 -4100 6100
+Connection ~ -4100 6100
+Wire Wire Line
+	-4100 6100 -4000 6100
+$Comp
+L power:+3.3VA #PWR?
+U 1 1 60B31123
+P -3900 6100
+F 0 "#PWR?" H -3900 5950 50  0001 C CNN
+F 1 "+3.3VA" H -3885 6273 50  0000 C CNN
+F 2 "" H -3900 6100 50  0001 C CNN
+F 3 "" H -3900 6100 50  0001 C CNN
+	1    -3900 6100
+	1    0    0    -1
+$EndComp
+$Comp
+L power:+3.3V #PWR?
+U 1 1 60B319CC
+P -5200 6100
+F 0 "#PWR?" H -5200 5950 50  0001 C CNN
+F 1 "+3.3V" H -5185 6273 50  0000 C CNN
+F 2 "" H -5200 6100 50  0001 C CNN
+F 3 "" H -5200 6100 50  0001 C CNN
+	1    -5200 6100
+	1    0    0    -1
+$EndComp
+Connection ~ -5200 6100
+Text GLabel -5800 6700 0    50   Input ~ 0
+BOOT0
+Text GLabel -5800 6400 0    50   Input ~ 0
+NRST
+$Comp
+L Device:C_Small C?
+U 1 1 60B5079F
+P -6700 7100
+F 0 "C?" H -6608 7146 50  0000 L CNN
+F 1 "2.2u" H -6608 7055 50  0000 L CNN
+F 2 "Capacitor_SMD:C_0603_1608Metric" H -6700 7100 50  0001 C CNN
+F 3 "~" H -6700 7100 50  0001 C CNN
+	1    -6700 7100
+	1    0    0    -1
+$EndComp
+$Comp
+L Device:C_Small C?
+U 1 1 60B507A5
+P -6350 7100
+F 0 "C?" H -6258 7146 50  0000 L CNN
+F 1 "2.2u" H -6258 7055 50  0000 L CNN
+F 2 "Capacitor_SMD:C_0603_1608Metric" H -6350 7100 50  0001 C CNN
+F 3 "~" H -6350 7100 50  0001 C CNN
+	1    -6350 7100
+	1    0    0    -1
+$EndComp
+$Comp
+L power:GND #PWR?
+U 1 1 60B507AB
+P -6700 7200
+F 0 "#PWR?" H -6700 6950 50  0001 C CNN
+F 1 "GND" H -6695 7027 50  0000 C CNN
+F 2 "" H -6700 7200 50  0001 C CNN
+F 3 "" H -6700 7200 50  0001 C CNN
+	1    -6700 7200
+	1    0    0    -1
+$EndComp
+$Comp
+L power:GND #PWR?
+U 1 1 60B507B1
+P -6350 7200
+F 0 "#PWR?" H -6350 6950 50  0001 C CNN
+F 1 "GND" H -6345 7027 50  0000 C CNN
+F 2 "" H -6350 7200 50  0001 C CNN
+F 3 "" H -6350 7200 50  0001 C CNN
+	1    -6350 7200
+	1    0    0    -1
+$EndComp
+Wire Wire Line
+	-6350 7000 -5800 7000
+Wire Wire Line
+	-5800 6900 -6700 6900
+Wire Wire Line
+	-6700 6900 -6700 7000
+Wire Wire Line
+	-5000 13300 -4900 13300
+Connection ~ -4900 13300
+Wire Wire Line
+	-4900 13300 -4800 13300
+Connection ~ -4800 13300
+Wire Wire Line
+	-4800 13300 -4700 13300
+Connection ~ -4700 13300
+Wire Wire Line
+	-4700 13300 -4600 13300
+Connection ~ -4600 13300
+Wire Wire Line
+	-4600 13300 -4500 13300
+Connection ~ -4500 13300
+Wire Wire Line
+	-4500 13300 -4400 13300
+Connection ~ -4400 13300
+Wire Wire Line
+	-4400 13300 -4300 13300
+Connection ~ -4300 13300
+Wire Wire Line
+	-4300 13300 -4200 13300
+Connection ~ -4200 13300
+Wire Wire Line
+	-4200 13300 -4100 13300
+$Comp
+L power:GND #PWR?
+U 1 1 60BB23E2
+P -4600 13300
+F 0 "#PWR?" H -4600 13050 50  0001 C CNN
+F 1 "GND" H -4550 13150 50  0000 C CNN
+F 2 "" H -4600 13300 50  0001 C CNN
+F 3 "" H -4600 13300 50  0001 C CNN
+	1    -4600 13300
+	1    0    0    -1
+$EndComp
+$Comp
+L power:+3.3VA #PWR?
+U 1 1 60BD708E
+P -5800 7100
+F 0 "#PWR?" H -5800 6950 50  0001 C CNN
+F 1 "+3.3VA" V -5900 7200 50  0000 C CNN
+F 2 "" H -5800 7100 50  0001 C CNN
+F 3 "" H -5800 7100 50  0001 C CNN
+	1    -5800 7100
+	0    -1   -1   0
+$EndComp
 $EndSCHEMATC

Commit message: Working on PCB design.
Parts:
- removed C22, C23: 2.2u, Capacitor_SMD:C_0603_1608Metric, symbol Device:C_Small
- removed U1: STM32F405RGT6, Package_QFP:LQFP-64_10x10mm_P0.5mm, symbol MCU_ST_STM32F4:STM32F405RGTx
- removed U?: STM32F429ZITx, Package_QFP:LQFP-144_20x20mm_P0.5mm, symbol MCU_ST_STM32F4:STM32F429ZITx
- added D?: RED, LED_SMD:LED_0603_1608Metric, symbol Device:LED_Small
- added D?: GREEN, LED_SMD:LED_0603_1608Metric, symbol Device:LED_Small
- added Q? (x2): Q_NPN_BCE, Package_TO_SOT_SMD:SOT-23, symbol Device:Q_NPN_BCE
- added R19, R20, R5: 10k, Resistor_SMD:R_0402_1005Metric, symbol Device:R_Small
- added R? (x2): 33, Resistor_SMD:R_0402_1005Metric, symbol Device:R_Small
- added R? (x2): 470, Resistor_SMD:R_0603_1608Metric, symbol Device:R_Small
- added SW7: SW_SPDT, Button_Switch_SMD:SW_SPDT_PCM12, symbol Switch:SW_SPDT
- added U1: STM32F427VITx, Package_QFP:LQFP-100_14x14mm_P0.5mm, symbol MCU_ST_STM32F4:STM32F427VITx
- C25, C26: value 12p -> 20p
- X1: renamed from 16MHz_1; value Y200 -> 25MHZ
- gave numbers to parts that had none: 2
Connections:
- net labels added: LED4, LED5
- net labels removed: BT3N_Input, USB_CONN_D+, USB_CONN_D-
- wire segments 236 -> 229
- no-connect marks 25 -> 53
Other:
- moved on the sheet: C11, C12, C13, C22, C23, C24, C25, C26, C27, C28, C29, C30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

Commit message: Making progress with Updating the new schematic and footprints
Parts:
- removed J10: I2C1, TerminalBlock_MetzConnect:TerminalBlock_MetzConnect_Type086_RT03404HBLC_1x04_P3.81mm_Horizontal, symbol Connector:Screw_Terminal_01x04
- removed J2: RS485, TerminalBlock_MetzConnect:TerminalBlock_MetzConnect_Type086_RT03404HBLC_1x04_P3.81mm_Horizontal, symbol Connector:Screw_Terminal_01x04
- removed J7: USART1, TerminalBlock_MetzConnect:TerminalBlock_MetzConnect_Type086_RT03404HBLC_1x04_P3.81mm_Horizontal, symbol Connector:Screw_Terminal_01x04
- removed J8: TIMER, TerminalBlock_MetzConnect:TerminalBlock_MetzConnect_Type086_RT03404HBLC_1x04_P3.81mm_Horizontal, symbol Connector:Screw_Terminal_01x04
- removed J9: ADC, TerminalBlock_MetzConnect:TerminalBlock_MetzConnect_Type086_RT03404HBLC_1x04_P3.81mm_Horizontal, symbol Connector:Screw_Terminal_01x04
- added J10: USART1_2, symbol Waveform~Generator-cache:Connector_Screw_Terminal_01x02
- added J19: ADC_2, symbol Waveform~Generator-cache:Connector_Screw_Terminal_01x02
- added J2: RS485_1, symbol Waveform~Generator-cache:Connector_Screw_Terminal_01x02
- added J20: TIMER_1, symbol Waveform~Generator-cache:Connector_Screw_Terminal_01x02
- added J21: I2C1_1, symbol Waveform~Generator-cache:Connector_Screw_Terminal_01x02
- added J22: TIMER_2, symbol Waveform~Generator-cache:Connector_Screw_Terminal_01x02
- added J23: I2C1_2, symbol Waveform~Generator-cache:Connector_Screw_Terminal_01x02
- added J7: RS485_2, symbol Waveform~Generator-cache:Connector_Screw_Terminal_01x02
- added J8: USART1_1, symbol Waveform~Generator-cache:Connector_Screw_Terminal_01x02
- added J9: ADC_1, symbol Waveform~Generator-cache:Connector_Screw_Terminal_01x02
- gave numbers to parts that had none: 8
Other:
- moved on the sheet: R33, R34, U10, U11, U6, U7

Commit message: Working on PCB footprint placement
Parts:
- added R39: 120, Resistor_SMD:R_0603_1608Metric, symbol Device:R_Small
- C22, C23: footprint Capacitor_SMD:C_0603_1608Metric -> Capacitor_SMD:C_0402_1005Metric
- F1: value 250mA -> 300mA
- FB2: value 600 @ 600 MHz -> 600 @ 600MHz
- J10, J19, J2, J20, J21, J22, J23, J7, J8, J9: footprint (none) -> Extra Components:5mm Pitch, 2 Way Terminal Block
- J5: footprint TerminalBlock_MetzConnect:TerminalBlock_MetzConnect_Type086_RT03402HBLC_1x02_P3.81mm_Horizontal -> Extra Components:5mm Pitch, 2 Way Terminal Block
- U2: value MAX485E -> MAX485EESAT
Connections:
- wire segments 229 -> 233
Other:
- moved on the sheet: C1, C10, C11, C12, C13, C2, C22, C23, C24, C25, C26, C27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

Commit message: Making progress with PCB layout
Changed lines of the file:
@@
-$EndComp
-$Comp
-L power:+5V #PWR0180
-U 1 1 604DF6A5
-P 7500 7150
-F 0 "#PWR0180" H 7500 7000 50  0001 C CNN
-F 1 "+5V" H 7515 7323 50  0000 C CNN
-F 2 "" H 7500 7150 50  0001 C CNN
-F 3 "" H 7500 7150 50  0001 C CNN
-	1    7500 7150
-	0    1    1    0
 $EndComp
 $Comp
@@
 Wire Wire Line
 	14650 2650 14800 2650
+$Comp
+L power:VBUS #PWR?
+U 1 1 61F8C500
+P 7500 7150
+F 0 "#PWR?" H 7500 7000 50  0001 C CNN
+F 1 "VBUS" H 7515 7323 50  0000 C CNN
+F 2 "" H 7500 7150 50  0001 C CNN
+F 3 "" H 7500 7150 50  0001 C CNN
+	1    7500 7150
+	0    1    -1   0
+$EndComp
 $EndSCHEMATC

Commit message: Working on PCB layout
Parts:
- J12: footprint TerminalBlock_MetzConnect:TerminalBlock_MetzConnect_Type086_RT03402HBLC_1x02_P3.81mm_Horizontal -> Extra Components:5mm Pitch, 2 Way Terminal Block
- J5: value Signal 2 -> Signal 1
Other:
- moved on the sheet: C27, C28, C29, C30, R1, R15, R16, R17, R18, R2, R3, R4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

Commit message: Updating PCB layout
Parts:
- added D11: BLUE, LED_SMD:LED_0603_1608Metric, symbol Device:LED_Small
- R10: value 1k -> 470
Connections:
- wire segments 233 -> 234
- no-connect marks 53 -> 54
Other:
- moved on the sheet: Q1, R11
Changed lines of the file:
@@
 Text GLabel 13800 2450 0    50   Input ~ 0
 RE
-Connection ~ 12400 2450
-Wire Wire Line
-	12400 2350 12400 2450
-$Comp
-L Device:Q_NPN_BCE Q1
-U 1 1 60EC531A
-P 12600 2450
-F 0 "Q1" H 12791 2496 50  0000 L CNN
-F 1 "Q_NPN_BCE" H 12791 2405 50  0000 L CNN
-F 2 "Package_TO_SOT_SMD:SOT-23" H 12800 2550 50  0001 C CNN
-F 3 "~" H 12600 2450 50  0001 C CNN
-	1    12600 2450
-	1    0    0    -1
-$EndComp
-Wire Wire Line
-	12850 2250 12700 2250
-Connection ~ 12700 2250
-Wire Wire Line
-	12700 2250 12700 2100
-Text GLabel 12850 2250 2    50   Input ~ 0
-DE
-Text GLabel 12400 2350 1    50   Input ~ 0
-RE
-$Comp
-L power:GND #PWR0151
-U 1 1 60ECC493
-P 12700 2650
-F 0 "#PWR0151" H 12700 2400 50  0001 C CNN
-F 1 "GND" H 12800 2550 50  0000 C CNN
-F 2 "" H 12700 2650 50  0001 C CNN
-F 3 "" H 12700 2650 50  0001 C CNN
-	1    12700 2650
-	1    0    0    -1
-$EndComp
-Text GLabel 12200 2450 0    51   Input ~ 0
-MAX485_DE
 $Comp
 L power:+3.3V #PWR0152
@@
 P 12700 2000
 F 0 "R10" H 12759 2046 50  0000 L CNN
-F 1 "1k" H 12759 1955 50  0000 L CNN
+F 1 "470" H 12759 1955 50  0000 L CNN
 F 2 "Resistor_SMD:R_0603_1608Metric" H 12700 2000 50  0001 C CNN
 F 3 "~" H 12700 2000 50  0001 C CNN
 	1    12700 2000
 	1    0    0    -1
-$EndComp
-$Comp
-L Device:R_Small R11
-U 1 1 60EC8C3B
-P 12300 2450
-F 0 "R11" V 12104 2450 50  0000 C CNN
-F 1 "1k" V 12200 2450 50  0000 C CNN
-F 2 "Resistor_SMD:R_0402_1005Metric" H 12300 2450 50  0001 C CNN
-F 3 "~" H 12300 2450 50  0001 C CNN
-	1    12300 2450
-	0    1    1    0
 $EndComp
 $Comp
@@
 Text GLabel 3400 8000 2    50   Input ~ 0
 USART1_RX
-Text GLabel 3400 7700 2    47   Input ~ 0
-SWDIO
 Text GLabel 3400 7000 2    47   Input ~ 0
 SWCLK
@@
 	0    1    -1   0
 $EndComp
+Wire Wire Line
+	12700 2100 12700 2150
+$Comp
+L Device:LED_Small D11
+U 1 1 62355C03
+P 12700 2250
+F 0 "D11" V 12746 2182 50  0000 R CNN
+F 1 "BLUE" V 12655 2182 50  0000 R CNN
+F 2 "LED_SMD:LED_0603_1608Metric" V 12700 2250 50  0001 C CNN
+F 3 "~" V 12700 2250 50  0001 C CNN
+	1    12700 2250
+	0    -1   -1   0
+$EndComp
+$Comp
+L Device:R_Small R11
+U 1 1 60EC8C3B
+P 12300 2750
+F 0 "R11" V 12104 2750 50  0000 C CNN
+F 1 "1k" V 12200 2750 50  0000 C CNN
+F 2 "Resistor_SMD:R_0402_1005Metric" H 12300 2750 50  0001 C CNN
+F 3 "~" H 12300 2750 50  0001 C CNN
+	1    12300 2750
+	0    1    1    0
+$EndComp
+Text GLabel 12200 2750 0    51   Input ~ 0
+MAX485_DE
+$Comp
+L power:GND #PWR0151
+U 1 1 60ECC493
+P 12700 2950
+F 0 "#PWR0151" H 12700 2700 50  0001 C CNN
+F 1 "GND" H 12800 2850 50  0000 C CNN
+F 2 "" H 12700 2950 50  0001 C CNN
+F 3 "" H 12700 2950 50  0001 C CNN
+	1    12700 2950
+	1    0    0    -1
+$EndComp
+Text GLabel 12400 2650 1    50   Input ~ 0
+RE
+Text GLabel 12850 2550 2    50   Input ~ 0
+DE
+Wire Wire Line
+	12850 2550 12700 2550
+$Comp
+L Device:Q_NPN_BCE Q1
+U 1 1 60EC531A
+P 12600 2750
+F 0 "Q1" H 12791 2796 50  0000 L CNN
+F 1 "Q_NPN_BCE" H 12791 2705 50  0000 L CNN
+F 2 "Package_TO_SOT_SMD:SOT-23" H 12800 2850 50  0001 C CNN
+F 3 "~" H 12600 2750 50  0001 C CNN
+	1    12600 2750
+	1    0    0    -1
+$EndComp
+Wire Wire Line
+	12400 2650 12400 2750
+Connection ~ 12400 2750
+Connection ~ 12700 2550
+Wire Wire Line
+	12700 2350 12700 2550
+NoConn ~ 3400 7700
 $EndSCHEMATC
