File: PCB/Waveform Generator/_autosave-Waveform Generator.sch (KiCad schematic (older format))
At the start: 115 parts, among them J1 12V Power, J10 Conn_01x04, J2 RS485, J3 USB_B_Micro, J4 Conn_01x02, J5 Conn_01x02, J6 SWD, J7 Conn_01x04, J8 Conn_01x04, J9 Conn_01x04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

Commit message: update
Parts:
- removed J1: 12V Power, symbol Connector_Generic:Conn_01x02
- removed J10, J7, J8, J9: Conn_01x04, symbol Connector_Generic:Conn_01x04
- removed J2: RS485, symbol Connector_Generic:Conn_01x04
- removed J4, J5: Conn_01x02, symbol Connector_Generic:Conn_01x02
- added J1: Power input, symbol Connector:Screw_Terminal_01x02
- added J10: I2C1, symbol Connector:Screw_Terminal_01x04
- added J2: RS485, symbol Connector:Screw_Terminal_01x04
- added J4: Signal 1, symbol Connector:Screw_Terminal_01x02
- added J5: Signal 2, symbol Connector:Screw_Terminal_01x02
- added J7: USART1, symbol Connector:Screw_Terminal_01x04
- added J8: TIMER, symbol Connector:Screw_Terminal_01x04
- added J9: ADC, symbol Connector:Screw_Terminal_01x04
- renumbered D7 to D8
Changed lines of the file:
@@
 DAC_OUT2
-$Comp
-L Connector_Generic:Conn_01x04 J7
-U 1 1 6072C1BC
-P 13900 8500
-F 0 "J7" H 13980 8492 50  0000 L CNN
-F 1 "Conn_01x04" H 13980 8401 50  0000 L CNN
-F 2 "" H 13900 8500 50  0001 C CNN
-F 3 "~" H 13900 8500 50  0001 C CNN
-	1    13900 8500
-	1    0    0    -1
-$EndComp
 $Comp
 L power:GND #PWR0128
@@
 ADC1_IN1
 $Comp
-L Connector_Generic:Conn_01x04 J9
-U 1 1 60730A09
-P 13850 9400
-F 0 "J9" H 13930 9392 50  0000 L CNN
-F 1 "Conn_01x04" H 13930 9301 50  0000 L CNN
-F 2 "" H 13850 9400 50  0001 C CNN
-F 3 "~" H 13850 9400 50  0001 C CNN
-	1    13850 9400
-	1    0    0    -1
-$EndComp
-$Comp
 L power:GND #PWR0130
 U 1 1 60730A0F
@@
 Text GLabel 2900 9650 2    51   Input ~ 0
 I2C1_SCL
-$Comp
-L Connector_Generic:Conn_01x04 J10
-U 1 1 6073F42F
-P 15300 9400
-F 0 "J10" H 15380 9392 50  0000 L CNN
-F 1 "Conn_01x04" H 15380 9301 50  0000 L CNN
-F 2 "" H 15300 9400 50  0001 C CNN
-F 3 "~" H 15300 9400 50  0001 C CNN
-	1    15300 9400
-	1    0    0    -1
-$EndComp
 $Comp
 L power:GND #PWR0132
@@
 Text GLabel 15050 8450 0    51   Input ~ 0
 TIM1_CH1
-$Comp
-L Connector_Generic:Conn_01x04 J8
-U 1 1 60767E94
-P 15250 8450
-F 0 "J8" H 15330 8442 50  0000 L CNN
-F 1 "Conn_01x04" H 15330 8351 50  0000 L CNN
-F 2 "" H 15250 8450 50  0001 C CNN
-F 3 "~" H 15250 8450 50  0001 C CNN
-	1    15250 8450
-	1    0    0    -1
-$EndComp
 $Comp
 L power:GND #PWR0134
@@
 	1    2250 1750
 	1    0    0    1
-$EndComp
-$Comp
-L Connector_Generic:Conn_01x02 J1
-U 1 1 604CA7F0
-P 1150 1750
-F 0 "J1" H 1250 1450 50  0000 C CNN
-F 1 "12V Power" H 1250 1550 50  0000 C CNN
-F 2 "" H 1150 1750 50  0001 C CNN
-F 3 "~" H 1150 1750 50  0001 C CNN
-	1    1150 1750
-	-1   0    0    1
 $EndComp
 $Comp
@@
 	1    0    0    -1
 $EndComp
-$Comp
-L Connector_Generic:Conn_01x04 J2
-U 1 1 60E54529
-P 15250 2450
-F 0 "J2" H 15330 2442 50  0000 L CNN
-F 1 "RS485" H 15330 2351 50  0000 L CNN
-F 2 "" H 15250 2450 50  0001 C CNN
-F 3 "~" H 15250 2450 50  0001 C CNN
-	1    15250 2450
-	1    0    0    -1
-$EndComp
 Text GLabel 13850 2350 0    50   Input ~ 0
 USART2_RX
@@
 $EndComp
 $Comp
-L Connector_Generic:Conn_01x02 J5
-U 1 1 605B4C62
-P 9550 8950
-F 0 "J5" H 9630 8942 50  0000 L CNN
-F 1 "Conn_01x02" H 9630 8851 50  0000 L CNN
-F 2 "" H 9550 8950 50  0001 C CNN
-F 3 "~" H 9550 8950 50  0001 C CNN
-	1    9550 8950
-	1    0    0    -1
-$EndComp
-$Comp
-L Connector_Generic:Conn_01x02 J4
-U 1 1 605A009D
-P 9550 7500
-F 0 "J4" H 9630 7492 50  0000 L CNN
-F 1 "Conn_01x02" H 9630 7401 50  0000 L CNN
-F 2 "" H 9550 7500 50  0001 C CNN
-F 3 "~" H 9550 7500 50  0001 C CNN
-	1    9550 7500
-	1    0    0    -1
-$EndComp
-$Comp
 L power:GND #PWR0170
 U 1 1 605A00A9
@@
 	4500 9300 4500 9350
 Connection ~ 4500 9350
-Connection ~ 1350 1650
 Wire Wire Line
 	2000 7150 2100 7150
@@
 $EndComp
 $Comp
-L power:GND #PWR?
+L power:GND #PWR0182
 U 1 1 615EC6D4
 P 10350 1900
-F 0 "#PWR?" H 10350 1650 50  0001 C CNN
+F 0 "#PWR0182" H 10350 1650 50  0001 C CNN
 F 1 "GND" H 10355 1727 50  0000 C CNN
 F 2 "" H 10350 1900 50  0001 C CNN
@@
 $EndComp
 $Comp
-L Device:LED_Small D7
+L Device:LED_Small D8
 U 1 1 615EC6DA
 P 10350 1600
-F 0 "D7" V 10396 1532 50  0000 R CNN
+F 0 "D8" V 10396 1532 50  0000 R CNN
 F 1 "GREEN" V 10305 1532 50  0000 R CNN
 F 2 "" V 10350 1600 50  0001 C CNN
@@
 Wire Notes Line
 	700  750  10800 750
+$Comp
+L Connector:Screw_Terminal_01x02 J1
+U 1 1 61627931
+P 1150 1750
+F 0 "J1" H 1200 1450 50  0000 C CNN
+F 1 "Power input" H 1250 1550 50  0000 C CNN
+F 2 "" H 1150 1750 50  0001 C CNN
+F 3 "~" H 1150 1750 50  0001 C CNN
+	1    1150 1750
+	-1   0    0    1
+$EndComp
+Connection ~ 1350 1650
+$Comp
+L Connector:Screw_Terminal_01x04 J2
+U 1 1 61629C36
+P 15250 2450
+F 0 "J2" H 15330 2442 50  0000 L CNN
+F 1 "RS485" H 15330 2351 50  0000 L CNN
+F 2 "" H 15250 2450 50  0001 C CNN
+F 3 "~" H 15250 2450 50  0001 C CNN
+	1    15250 2450
+	1    0    0    -1
+$EndComp
+$Comp
+L Connector:Screw_Terminal_01x02 J4
+U 1 1 6162CC34
+P 9550 7500
+F 0 "J4" H 9630 7492 50  0000 L CNN
+F 1 "Signal 1" H 9630 7401 50  0000 L CNN
+F 2 "" H 9550 7500 50  0001 C CNN
+F 3 "~" H 9550 7500 50  0001 C CNN
+	1    9550 7500
+	1    0    0    -1
+$EndComp
+$Comp
+L Connector:Screw_Terminal_01x02 J5
+U 1 1 6162DCDE
+P 9550 8950
+F 0 "J5" H 9630 8942 50  0000 L CNN
+F 1 "Signal 2" H 9630 8851 50  0000 L CNN
+F 2 "" H 9550 8950 50  0001 C CNN
+F 3 "~" H 9550 8950 50  0001 C CNN
+	1    9550 8950
+	1    0    0    -1
+$EndComp
+$Comp
+L Connector:Screw_Terminal_01x04 J7
+U 1 1 6162F55F
+P 13900 8500
+F 0 "J7" H 13980 8492 50  0000 L CNN
+F 1 "USART1" H 13980 8401 50  0000 L CNN
+F 2 "" H 13900 8500 50  0001 C CNN
+F 3 "~" H 13900 8500 50  0001 C CNN
+	1    13900 8500
+	1    0    0    -1
+$EndComp
+$Comp
+L Connector:Screw_Terminal_01x04 J10
+U 1 1 61630A48
+P 15300 9400
+F 0 "J10" H 15380 9392 50  0000 L CNN
+F 1 "I2C1" H 15380 9301 50  0000 L CNN
+F 2 "" H 15300 9400 50  0001 C CNN
+F 3 "~" H 15300 9400 50  0001 C CNN
+	1    15300 9400
+	1    0    0    -1
+$EndComp
+$Comp
+L Connector:Screw_Terminal_01x04 J8
+U 1 1 616310F5
+P 15250 8450
+F 0 "J8" H 15330 8442 50  0000 L CNN
+F 1 "TIMER" H 15330 8351 50  0000 L CNN
+F 2 "" H 15250 8450 50  0001 C CNN
+F 3 "~" H 15250 8450 50  0001 C CNN
+	1    15250 8450
+	1    0    0    -1
+$EndComp
+$Comp
+L Connector:Screw_Terminal_01x04 J9
+U 1 1 6163141B
+P 13850 9400
+F 0 "J9" H 13930 9392 50  0000 L CNN
+F 1 "ADC" H 13930 9301 50  0000 L CNN
+F 2 "" H 13850 9400 50  0001 C CNN
+F 3 "~" H 13850 9400 50  0001 C CNN
+	1    13850 9400
+	1    0    0    -1
+$EndComp
 $EndSCHEMATC

Commit message: Updating Schematic
Parts:
- added U8: LM335ADT, symbol Extra~Components:LM335ADT
Changed lines of the file:
@@
+	1    0    0    -1
+$EndComp
+$Comp
+L Extra~Components:LM335ADT U8
+U 1 1 6164C72A
+P 11650 5100
+F 0 "U8" H 11625 5536 59  0000 C CNN
+F 1 "LM335ADT" H 11625 5431 59  0000 C CNN
+F 2 "" V 11500 5050 59  0001 C CNN
+F 3 "" V 11500 5050 59  0001 C CNN
+	1    11650 5100
+	1    0    0    -1
+$EndComp
+$Comp
+L power:GND #PWR?
+U 1 1 6164F24E
+P 12100 4950
+F 0 "#PWR?" H 12100 4700 50  0001 C CNN
+F 1 "GND" H 12105 4777 50  0000 C CNN
+F 2 "" H 12100 4950 50  0001 C CNN
+F 3 "" H 12100 4950 50  0001 C CNN
+	1    12100 4950
 	1    0    0    -1
 $EndComp
