File: PCB/Waveform Generator/_autosave-Waveform Generator.sch (KiCad schematic (older format))
At the start: 122 parts, among them J1 Power input, J10 I2C1, J11 5001, J12 Signal 2, J13 5001, J14 5001, J15 5001, J16 5001, J17 5001, J18 5001, J2 RS485, J3 USB_B_Micro, J4 5001, J5 Signal 2, J6 SWD, J7 USART1, J8 TIMER, J9 ADC, Q0 AO3401A, Q1 Q_NPN_BCE, Q2 Q_NPN_BCE, Q3 Q_PNP_BCE, Q4 Q_NPN_BCE, Q5 Q_NPN_BCE, Q6 Q_NPN_BCE, SW1 SW_SPDT, SW2 RESET Button, SW3 SW_SPDT, SW4 Btn1, SW5 Btn1, SW6 Btn1, U1 STM32F405RGT6, U2 MAX485E, U3 USBLC6-2SC6, U4 LTC2051HVIMS8, U5 LTC2051HVIMS8, U8 LM335ADT

Commit message: Working
Parts:
- added D8: GREEN, LED_SMD:LED_0603_1608Metric, symbol Device:LED_Small
- added R35: 1k, Resistor_SMD:R_0603_1608Metric, symbol Device:R_Small
- added U?: STM32F439ZITx, Package_QFP:LQFP-144_20x20mm_P0.5mm, symbol MCU_ST_STM32F4:STM32F439ZITx
- PS1: value ITP0312D05 -> ITP0324D05
Changed lines of the file:
@@
 	8750 1700 8750 1600
-$Comp
-L Device:R_Small R6
-U 1 1 60360DB4
-P 9550 2000
-F 0 "R6" H 9609 2046 50  0000 L CNN
-F 1 "1k" H 9609 1955 50  0000 L CNN
-F 2 "Resistor_SMD:R_0603_1608Metric" H 9550 2000 50  0001 C CNN
-F 3 "~" H 9550 2000 50  0001 C CNN
-	1    9550 2000
-	1    0    0    -1
-$EndComp
-$Comp
-L power:GND #PWR0127
-U 1 1 60361815
-P 9550 2100
-F 0 "#PWR0127" H 9550 1850 50  0001 C CNN
-F 1 "GND" H 9555 1927 50  0000 C CNN
-F 2 "" H 9550 2100 50  0001 C CNN
-F 3 "" H 9550 2100 50  0001 C CNN
-	1    9550 2100
-	1    0    0    -1
-$EndComp
 $Comp
 L Switch:SW_SPDT SW1
@@
 $EndComp
 NoConn ~ 10150 1700
-Wire Wire Line
-	9550 1600 9550 1700
-$Comp
-L Device:LED_Small D3
-U 1 1 6035F732
-P 9550 1800
-F 0 "D3" V 9596 1732 50  0000 R CNN
-F 1 "GREEN" V 9505 1732 50  0000 R CNN
-F 2 "LED_SMD:LED_0603_1608Metric" V 9550 1800 50  0001 C CNN
-F 3 "~" V 9550 1800 50  0001 C CNN
-	1    9550 1800
-	0    -1   -1   0
-$EndComp
 Text Notes 5600 1250 0    47   ~ 0
 5v to 3v3\n
 Connection ~ 8750 1600
-Wire Wire Line
-	9550 1600 9750 1600
-Connection ~ 9550 1600
 Text Notes 9350 1250 0    47   ~ 0
 Pwr LED and Switch
@@
 P 2900 1800
 F 0 "PS1" H 2900 2200 59  0000 C CNN
-F 1 "ITP0312D05" H 2900 2100 59  0000 C CNN
+F 1 "ITP0324D05" H 2900 2100 59  0000 C CNN
 F 2 "Extra Components:ITP0312D05" H 3100 1800 59  0001 C CNN
 F 3 "" H 3100 1800 59  0001 C CNN
@@
 	8850 1600 8850 1500
 Connection ~ 8850 1600
-Wire Wire Line
-	8850 1600 9550 1600
 $Comp
 L Extra~Components:5001 J17
@@
 Wire Notes Line
 	6400 9250 6400 6400
+Wire Wire Line
+	8850 1600 9550 1600
+Wire Wire Line
+	9550 1600 9750 1600
+Connection ~ 9550 1600
+Wire Wire Line
+	9550 1600 9550 1700
+$Comp
+L Device:LED_Small D3
+U 1 1 6035F732
+P 9550 1800
+F 0 "D3" V 9596 1732 50  0000 R CNN
+F 1 "GREEN" V 9505 1732 50  0000 R CNN
+F 2 "LED_SMD:LED_0603_1608Metric" V 9550 1800 50  0001 C CNN
+F 3 "~" V 9550 1800 50  0001 C CNN
+	1    9550 1800
+	0    -1   -1   0
+$EndComp
+$Comp
+L power:GND #PWR0127
+U 1 1 60361815
+P 9550 2100
+F 0 "#PWR0127" H 9550 1850 50  0001 C CNN
+F 1 "GND" H 9555 1927 50  0000 C CNN
+F 2 "" H 9550 2100 50  0001 C CNN
+F 3 "" H 9550 2100 50  0001 C CNN
+	1    9550 2100
+	1    0    0    -1
+$EndComp
+$Comp
+L Device:R_Small R6
+U 1 1 60360DB4
+P 9550 2000
+F 0 "R6" H 9609 2046 50  0000 L CNN
+F 1 "1k" H 9609 1955 50  0000 L CNN
+F 2 "Resistor_SMD:R_0603_1608Metric" H 9550 2000 50  0001 C CNN
+F 3 "~" H 9550 2000 50  0001 C CNN
+	1    9550 2000
+	1    0    0    -1
+$EndComp
+$Comp
+L Device:LED_Small D8
+U 1 1 6031020B
+P 4350 1700
+F 0 "D8" V 4396 1632 50  0000 R CNN
+F 1 "GREEN" V 4305 1632 50  0000 R CNN
+F 2 "LED_SMD:LED_0603_1608Metric" V 4350 1700 50  0001 C CNN
+F 3 "~" V 4350 1700 50  0001 C CNN
+	1    4350 1700
+	0    -1   -1   0
+$EndComp
+$Comp
+L power:GND #PWR?
+U 1 1 60310211
+P 4350 2000
+F 0 "#PWR?" H 4350 1750 50  0001 C CNN
+F 1 "GND" H 4355 1827 50  0000 C CNN
+F 2 "" H 4350 2000 50  0001 C CNN
+F 3 "" H 4350 2000 50  0001 C CNN
+	1    4350 2000
+	1    0    0    -1
+$EndComp
+$Comp
+L Device:R_Small R35
+U 1 1 60310217
+P 4350 1900
+F 0 "R35" H 4409 1946 50  0000 L CNN
+F 1 "1k" H 4409 1855 50  0000 L CNN
+F 2 "Resistor_SMD:R_0603_1608Metric" H 4350 1900 50  0001 C CNN
+F 3 "~" H 4350 1900 50  0001 C CNN
+	1    4350 1900
+	1    0    0    -1
+$EndComp
+$Comp
+L MCU_ST_STM32F4:STM32F439ZITx U?
+U 1 1 6031F6E7
+P -6450 8600
+F 0 "U?" H -6450 4911 50  0000 C CNN
+F 1 "STM32F439ZITx" H -6450 4820 50  0000 C CNN
+F 2 "Package_QFP:LQFP-144_20x20mm_P0.5mm" H -7450 5200 50  0001 R CNN
+F 3 "http://www.st.com/st-web-ui/static/active/en/resource/technical/document/datasheet/DM00077036.pdf" H -6450 8600 50  0001 C CNN
+	1    -6450 8600
+	1    0    0    -1
+$EndComp
 $EndSCHEMATC
