File: PCB/Waveform Generator/_autosave-Waveform Generator.sch (KiCad schematic (older format))
At the start: 141 parts, among them J1 Power input, J10 USART1_2, J12 Signal 2, J19 ADC_2, J2 RS485_1, J20 TIMER_1, J21 I2C1_1, J22 TIMER_2, J23 I2C1_2, J3 USB_B_Micro, J5 Signal 1, J6 SWD, J7 RS485_2, J8 USART1_1, J9 ADC_1, Q0 AO3401A, Q1 Q_NPN_BCE, Q2 Q_NPN_BCE, Q3 Q_PNP_BCE, Q4 Q_NPN_BCE, Q5 Q_NPN_BCE, Q6 Q_NPN_BCE, Q7 Q_NPN_BCE, Q8 Q_NPN_BCE, SW1 SW_SPDT, SW2 SW_SPDT, SW3 SW_SPDT, T0 GND, T1 5V, T2 3V3, T3 5001, T5 RS485_A, T6 DAC_OUT_2, T7 DAC_OUT_1, U1 STM32F427VITx, U10 USBLC6-2SC6, U11 USBLC6-2SC6, U2 MAX485EESAT, U3 USBLC6-2SC6, U4 OPA1602, U5 OPA1602, U6 USBLC6-2SC6, U7 USBLC6-2SC6, U8 LM335ADT, U9 USBLC6-2SC6, X1 25MHZ

Commit message: Adding markers to indicator pin 1
Parts:
- 3V3: renamed from T2; value 3V3 -> 5001
- 5V1: renamed from T1; value 5V -> 5001
- DAC_OUT_1: renamed from T7; value DAC_OUT_1 -> 5001
- DAC_OUT_2: renamed from T6; value DAC_OUT_2 -> 5001
- GND1: renamed from T0; value GND -> 5001
- RS485_A1: renamed from T5; value RS485_A -> 5001
- renumbered RS485_B to RS485_B1, T3 to TEMP_SENSE
Changed lines of the file:
@@
 	0    -1   -1   0
 $EndComp
-$Comp
-L Extra~Components:5001 RS485_B
-U 1 1 602D06EE
-P 14950 1900
-F 0 "RS485_B" H 15028 1908 59  0000 L CNN
-F 1 "5001" H 15028 1803 59  0000 L CNN
-F 2 "Extra Components:5001 Test Point" H 15000 1850 59  0001 C CNN
-F 3 "" H 15000 1850 59  0001 C CNN
-	1    14950 1900
-	1    0    0    -1
-$EndComp
 Wire Wire Line
 	14800 2450 15000 2450
@@
 	14800 2550 15000 2550
 $Comp
-L Extra~Components:5001 T1
-U 1 1 6030FC76
-P 5300 1900
-F 0 "T1" H 5400 2150 59  0000 C CNN
-F 1 "5V" H 5400 2050 59  0000 C CNN
-F 2 "Extra Components:5001 Test Point" H 5350 1850 59  0001 C CNN
-F 3 "" H 5350 1850 59  0001 C CNN
-	1    5300 1900
-	-1   0    0    1
-$EndComp
-$Comp
-L Extra~Components:5001 T2
-U 1 1 60330D7E
-P 7200 1400
-F 0 "T2" H 7142 1064 59  0000 C CNN
-F 1 "3V3" H 7142 1169 59  0000 C CNN
-F 2 "Extra Components:5001 Test Point" H 7250 1350 59  0001 C CNN
-F 3 "" H 7250 1350 59  0001 C CNN
-	1    7200 1400
-	0    -1   -1   0
-$EndComp
-$Comp
-L Extra~Components:5001 T3
+L Extra~Components:5001 TEMP_SENSE
 U 1 1 6035F161
 P 6700 4900
-F 0 "T3" H 6900 4800 59  0000 C CNN
+F 0 "TEMP_SENSE" H 6900 4800 59  0000 C CNN
 F 1 "5001" H 6900 4900 59  0000 C CNN
 F 2 "Extra Components:5001 Test Point" H 6750 4850 59  0001 C CNN
@@
 Wire Notes Line
 	6250 4200 7950 4200
-$Comp
-L Extra~Components:5001 T0
-U 1 1 603B19CE
-P 13000 5850
-F 0 "T0" H 13200 5750 59  0000 C CNN
-F 1 "GND" H 13200 5850 59  0000 C CNN
-F 2 "Extra Components:5001 Test Point" H 13050 5800 59  0001 C CNN
-F 3 "" H 13050 5800 59  0001 C CNN
-	1    13000 5850
-	1    0    0    -1
-$EndComp
 Wire Wire Line
 	12750 5550 12750 5850
@@
 $Comp
 L Amplifier_Operational:OPA1602 U4
-U 2 1 604A81A8
-P 8500 10000
-F 0 "U4" H 8300 10400 50  0000 C CNN
-F 1 "OPA1602" H 8300 10300 50  0000 C CNN
-F 2 "Package_SO:SOP-8_3.9x4.9mm_P1.27mm" H 8500 10000 50  0001 C CNN
-F 3 "http://www.ti.com/lit/ds/symlink/opa1604.pdf" H 8500 10000 50  0001 C CNN
-	2    8500 10000
-	1    0    0    -1
-$EndComp
-$Comp
-L Amplifier_Operational:OPA1602 U4
 U 3 1 604AB9C1
 P 8200 10650
@@
 Wire Wire Line
 	8800 10250 8800 10000
-$Comp
-L Extra~Components:5001 T7
-U 1 1 6085EE9A
-P 8800 9850
-F 0 "T7" V 9000 9800 59  0000 L CNN
-F 1 "DAC_OUT_1" V 8900 9600 59  0000 L CNN
-F 2 "Extra Components:5001 Test Point" H 8850 9800 59  0001 C CNN
-F 3 "" H 8850 9800 59  0001 C CNN
-	1    8800 9850
-	0    -1   -1   0
-$EndComp
 Connection ~ 8800 10000
 $Comp
@@
 $Comp
 L Amplifier_Operational:OPA1602 U5
-U 2 1 607192EF
-P 8500 8900
-F 0 "U5" H 8350 9250 50  0000 C CNN
-F 1 "OPA1602" H 8350 9150 50  0000 C CNN
-F 2 "Package_SO:SOP-8_3.9x4.9mm_P1.27mm" H 8500 8900 50  0001 C CNN
-F 3 "http://www.ti.com/lit/ds/symlink/opa1604.pdf" H 8500 8900 50  0001 C CNN
-	2    8500 8900
-	1    0    0    -1
-$EndComp
-$Comp
-L Amplifier_Operational:OPA1602 U5
 U 3 1 607192F5
 P 8100 8400
@@
 Wire Wire Line
 	8800 9150 8800 8900
-$Comp
-L Extra~Components:5001 T6
-U 1 1 60719318
-P 8800 8750
-F 0 "T6" V 9000 8700 59  0000 L CNN
-F 1 "DAC_OUT_2" V 8900 8500 59  0000 L CNN
-F 2 "Extra Components:5001 Test Point" H 8850 8700 59  0001 C CNN
-F 3 "" H 8850 8700 59  0001 C CNN
-	1    8800 8750
-	0    -1   -1   0
-$EndComp
 Connection ~ 8800 8900
 Text GLabel 6750 9100 0    51   Input ~ 0
@@
 NoConn ~ 15750 50
 $Comp
-L Extra~Components:5001 T5
-U 1 1 602D3514
-P 14950 3050
-F 0 "T5" H 15028 3058 59  0000 L CNN
-F 1 "RS485_A" H 15028 2953 59  0000 L CNN
-F 2 "Extra Components:5001 Test Point" H 15000 3000 59  0001 C CNN
-F 3 "" H 15000 3000 59  0001 C CNN
-	1    14950 3050
-	1    0    0    -1
-$EndComp
-$Comp
 L Switch:SW_Push BTN0
 U 1 1 6028E938
@@
 USART2_RTS
 NoConn ~ 3400 9100
+$Comp
+L Extra~Components:5001 GND1
+U 1 1 603B19CE
+P 13000 5850
+F 0 "GND1" H 13200 5750 59  0000 C CNN
+F 1 "5001" H 13200 5850 59  0000 C CNN
+F 2 "Extra Components:5001 Test Point" H 13050 5800 59  0001 C CNN
+F 3 "" H 13050 5800 59  0001 C CNN
+	1    13000 5850
+	1    0    0    -1
+$EndComp
+$Comp
+L Amplifier_Operational:OPA1602 U5
+U 2 1 607192EF
+P 8500 8900
+F 0 "U5" H 8500 9267 50  0000 C CNN
+F 1 "OPA1602" H 8500 9176 50  0000 C CNN
+F 2 "Package_SO:SOP-8_3.9x4.9mm_P1.27mm" H 8500 8900 50  0001 C CNN
+F 3 "http://www.ti.com/lit/ds/symlink/opa1604.pdf" H 8500 8900 50  0001 C CNN
+	2    8500 8900
+	1    0    0    -1
+$EndComp
+$Comp
+L Amplifier_Operational:OPA1602 U4
+U 2 1 604A81A8
+P 8500 10000
+F 0 "U4" H 8500 10367 50  0000 C CNN
+F 1 "OPA1602" H 8500 10276 50  0000 C CNN
+F 2 "Package_SO:SOP-8_3.9x4.9mm_P1.27mm" H 8500 10000 50  0001 C CNN
+F 3 "http://www.ti.com/lit/ds/symlink/opa1604.pdf" H 8500 10000 50  0001 C CNN
+	2    8500 10000
+	1    0    0    -1
+$EndComp
+$Comp
+L Extra~Components:5001 DAC_OUT_1
+U 1 1 6085EE9A
+P 8800 9850
+F 0 "DAC_OUT_1" V 9000 9600 59  0000 L CNN
+F 1 "5001" V 8900 9750 59  0000 L CNN
+F 2 "Extra Components:5001 Test Point" H 8850 9800 59  0001 C CNN
+F 3 "" H 8850 9800 59  0001 C CNN
+	1    8800 9850
+	0    -1   -1   0
+$EndComp
+$Comp
+L Extra~Components:5001 DAC_OUT_2
+U 1 1 60719318
+P 8800 8750
+F 0 "DAC_OUT_2" V 9000 8400 59  0000 L CNN
+F 1 "5001" V 8900 8650 59  0000 L CNN
+F 2 "Extra Components:5001 Test Point" H 8850 8700 59  0001 C CNN
+F 3 "" H 8850 8700 59  0001 C CNN
+	1    8800 8750
+	0    -1   -1   0
+$EndComp
+$Comp
+L Extra~Components:5001 RS485_A1
+U 1 1 602D3514
+P 14950 3050
+F 0 "RS485_A1" H 15028 3058 59  0000 L CNN
+F 1 "5001" H 15028 2953 59  0000 L CNN
+F 2 "Extra Components:5001 Test Point" H 15000 3000 59  0001 C CNN
+F 3 "" H 15000 3000 59  0001 C CNN
+	1    14950 3050
+	1    0    0    -1
+$EndComp
+$Comp
+L Extra~Components:5001 3V3
+U 1 1 60330D7E
+P 7200 1400
+F 0 "3V3" H 7142 1064 59  0000 C CNN
+F 1 "5001" H 7142 1169 59  0000 C CNN
+F 2 "Extra Components:5001 Test Point" H 7250 1350 59  0001 C CNN
+F 3 "" H 7250 1350 59  0001 C CNN
+	1    7200 1400
+	0    -1   -1   0
+$EndComp
+$Comp
+L Extra~Components:5001 5V1
+U 1 1 6030FC76
+P 5300 1900
+F 0 "5V1" H 5400 2150 59  0000 C CNN
+F 1 "5001" H 5400 2050 59  0000 C CNN
+F 2 "Extra Components:5001 Test Point" H 5350 1850 59  0001 C CNN
+F 3 "" H 5350 1850 59  0001 C CNN
+	1    5300 1900
+	-1   0    0    1
+$EndComp
+$Comp
+L Extra~Components:5001 RS485_B1
+U 1 1 602D06EE
+P 14950 1900
+F 0 "RS485_B1" H 15028 1908 59  0000 L CNN
+F 1 "5001" H 15028 1803 59  0000 L CNN
+F 2 "Extra Components:5001 Test Point" H 15000 1850 59  0001 C CNN
+F 3 "" H 15000 1850 59  0001 C CNN
+	1    14950 1900
+	1    0    0    -1
+$EndComp
 $EndSCHEMATC
