File: PCB/Waveform Generator/Waveform Generator.kicad_pcb (KiCad board)
At the start: 4 copper layers, 141 parts, among them J1 Power input, J10 USART1_2, J11 5001, J12 Signal 2, J13 5001, J14 5001, J15 5001, J16 5001, J17 5001, J18 5001, J19 ADC_2, J2 RS485_1, J20 TIMER_1, J21 I2C1_1, J22 TIMER_2, J23 I2C1_2, J3 USB_B_Micro, J4 5001, J5 Signal 1, J6 SWD, J7 RS485_2, J8 USART1_1, J9 ADC_1, Q0 AO3401A, Q1 Q_NPN_BCE, Q2 Q_NPN_BCE, Q3 Q_PNP_BCE, Q4 Q_NPN_BCE, Q5 Q_NPN_BCE, Q6 Q_NPN_BCE, Q7 Q_NPN_BCE, Q8 Q_NPN_BCE, SW1 SW_SPDT, SW2 RESET Button, SW3 SW_SPDT, SW4 Btn1, SW5 Btn1, SW6 Btn1, SW7 SW_SPDT, U1 STM32F427VITx, U10 USBLC6-2SC6, U11 USBLC6-2SC6, U2 MAX485EESAT, U3 USBLC6-2SC6, U4 OPA1602, U5 OPA1602, U6 USBLC6-2SC6, U7 USBLC6-2SC6, U8 LM335ADT, U9 USBLC6-2SC6, X1 25MHZ

Commit message: Working on PCB Layout
Parts:
- moved R28 100.3 mm to (46.6, 106.3), turned to 0 degrees
- moved R27 98.8 mm to (46.0, 98.0)
- moved D7 98.8 mm to (46.6, 104.7), turned to 0 degrees
- moved Q6 96.9 mm to (46.8, 100.4), turned to 0 degrees
- moved R26 91.2 mm to (52.5, 106.2)
- moved D6 89.9 mm to (52.4, 104.5), turned to 0 degrees
- moved R25 89.5 mm to (52.9, 98.0), turned to 180 degrees
- moved Q5 88.9 mm to (52.1, 100.3), turned to 0 degrees
- moved R5 60.7 mm to (75.2, 57.5), turned to 270 degrees
- moved SW7 55.4 mm to (78.4, 57.6), turned to 90 degrees
- moved R13 53.3 mm to (75.2, 48.8), turned to 270 degrees
- moved SW3 47.0 mm to (78.4, 48.2), turned to 90 degrees
- moved D5 15.0 mm to (120.8, 81.5)
- moved R23 15.0 mm to (123.3, 81.7)
- moved Q4 15.0 mm to (122.0, 84.0)
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
Commit message: Working on PCB design
Parts:
- J1: footprint TerminalBlock_MetzConnect:TerminalBlock_MetzConnect_Type086_RT03402HBLC_1x02_P3.81mm_Horizontal -> Extra Components:5mm Pitch, 2 Way Terminal Block
- moved D10 59.9 mm to (76.8, 41.0)
- moved D2 59.9 mm to (76.7, 32.9)
- moved R21 59.9 mm to (76.7, 31.2)
- moved R38 59.9 mm to (79.3, 41.4)
- moved Q7 59.9 mm to (78.0, 35.5)
- moved Q8 59.9 mm to (78.0, 43.6)
- moved R22 59.9 mm to (76.7, 39.5)
- moved R37 59.9 mm to (79.3, 33.1)
- moved D5 54.6 mm to (76.4, 49.6)
- moved Q4 54.6 mm to (77.6, 52.2)
- moved R23 54.6 mm to (79.0, 49.9)
- moved R24 54.6 mm to (76.5, 48.0)
- moved J1 25.8 mm to (36.0, 18.3)
- moved J16 25.8 mm to (72.8, 26.3)
- moved C3 25.5 mm to (49.5, 24.4)
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
Commit message: Making good progress
Parts:
- moved J3 11.6 mm to (89.8, 25.9), turned to 90 degrees
- moved R37 9.72 mm to (83.2, 42.0)
- moved R21 9.72 mm to (80.5, 40.1)
- moved D2 9.72 mm to (80.5, 41.8)
- moved Q7 9.72 mm to (81.8, 44.4)
- moved R14 9.36 mm to (58.5, 44.0), turned to 270 degrees
- moved U3 8.27 mm to (83.2, 30.7)
- moved R19 8.27 mm to (58.4, 41.8), turned to 90 degrees
- moved J6 7.95 mm to (60.4, 44.9), turned to 180 degrees
- moved U8 7.84 mm to (51.3, 33.9)
- moved Q8 7.36 mm to (73.3, 37.9)
- moved D10 7.36 mm to (72.2, 35.3)
- moved R22 7.36 mm to (72.1, 33.7)
- moved R38 7.36 mm to (74.7, 35.6)
- moved R29 6.89 mm to (64.2, 45.5), turned to 180 degrees
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
Commit message: Finalizing PCB layout
Parts:
- BTN2: renamed from SW5; value Btn1 -> Btn2
- BTN3: renamed from SW6; value Btn1 -> BTN3
- moved R33 4.83 mm to (39.0, 48.2), turned to 0 degrees
- moved C16 4.82 mm to (39.1, 41.4)
- moved C18 4.82 mm to (39.1, 44.1)
- moved C14 4.82 mm to (39.1, 38.7)
- moved C15 4.82 mm to (39.1, 40.0)
- moved C17 4.82 mm to (39.1, 42.7)
- moved C19 4.82 mm to (39.1, 45.4)
- moved R34 4.12 mm to (39.0, 49.4), turned to 0 degrees
- moved R36 1.43 mm to (51.5, 26.7), turned to 180 degrees
- moved R35 1.36 mm to (83.6, 20.3), turned to 0 degrees
- moved PWR1 1.13 mm to (51.6, 28.4), turned to 0 degrees
- moved R6 0.25 mm to (77.0, 20.3)
- moved PWR3 0.25 mm to (80.2, 20.3)
- moved LED2 0.12 mm to (67.1, 88.6)
- renumbered SW2 to BTN0, SW4 to BTN1, D7 to LED1, D6 to LED2, D5 to LED3, D10 to LED4, D2 to LED5, D9 to PWR1, D3 to PWR2, D8 to PWR3, SW7 to SW2, J18 to T0, J15 to T1, J16 to T2, J17 to T3, J13 to T4, J14 to T5, J11 to T6, J4 to T7

Commit message: Made good progress
Parts:
- moved H2 111.8 mm to (88.7, 15.6)
- moved H3 88.3 mm to (22.5, 105.1)
- moved H1 66.6 mm to (22.1, 15.4)
- moved Q4 13.5 mm to (79.3, 37.0)
- moved R38 12.8 mm to (81.7, 46.3), turned to 270 degrees
- moved R23 12.5 mm to (81.8, 36.3), turned to 270 degrees
- moved Q8 10.9 mm to (79.3, 47.1)
- moved R21 10.2 mm to (71.4, 44.6)
- moved LED5 10.2 mm to (71.4, 46.3)
- moved LED3 7.98 mm to (71.4, 39.7)
- moved R24 7.92 mm to (71.4, 38.1)
- moved LED4 7.74 mm to (71.4, 43.0)
- moved R22 7.74 mm to (71.4, 41.4)
- moved U7 3.96 mm to (38.3, 61.2)
- moved Q7 3.43 mm to (79.3, 42.0)
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
Commit message: Making progress
Parts:
- moved C21 7.06 mm to (49.9, 71.6), turned to 180 degrees
- moved C20 6.42 mm to (49.9, 72.8), turned to 0 degrees
- moved U7 3.76 mm to (38.5, 57.4)
- moved FB2 2.76 mm to (47.4, 72.1)
- moved C24 2.72 mm to (42.3, 68.1)
- moved H3 1.87 mm to (21.6, 106.7)
- moved SW1 1.81 mm to (78.2, 13.8)
- moved J1 1.57 mm to (39.1, 15.4)
- moved C7 1.53 mm to (71.0, 28.7)
- moved C8 1.53 mm to (71.0, 30.3)
- moved C9 1.53 mm to (71.0, 27.1)
- moved C10 1.53 mm to (71.0, 25.5)
- moved PS2 1.28 mm to (68.8, 15.0)
- moved PS1 1.17 mm to (55.0, 17.8)
- moved BTN0 0.86 mm to (39.2, 68.2), turned to 90 degrees
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Connections:
- R11 pad 2: MAX485_DE -> USART2_RTS
- U1 pad 16: MAX485_DE -> (no net)
- U1 pad 85: (no net) -> USART2_RTS
Other:
- board outline added: 80 x 104.1 mm
- board text added: "Waveform Generator v1 Nanodyn Systems"

Commit message: Making progress
Parts:
- moved C14 42.5 mm to (67.8, 70.0), turned to 0 degrees
- moved C16 35.1 mm to (71.8, 54.1), turned to 0 degrees
- moved C15 34.7 mm to (55.9, 70.4)
- moved C18 22.1 mm to (50.1, 63.3)
- moved C19 21.9 mm to (50.1, 64.4)
- moved C17 18.5 mm to (55.7, 50.8), turned to 0 degrees
- moved R33 14.5 mm to (50.8, 56.6)
- moved R34 14.4 mm to (50.8, 57.7)
- moved R12 2.81 mm to (47.0, 60.2), turned to 180 degrees
- moved R13 2.27 mm to (86.8, 36.2)
- moved C26 1.50 mm to (45.0, 60.8), turned to 0 degrees
- moved U10 0.44 mm to (73.3, 73.1)
- moved U7 0.28 mm to (38.2, 57.4)
- moved C25 0.27 mm to (44.0, 55.2)
Routing:
- net HSE_IN: track 0.00 -> 17.0 mm
- net GND: track 0.00 -> 10.1 mm, vias 0 -> 2
- net HSE_OUT: track 0.00 -> 6.07 mm
- net Net-(C26-Pad2): track 0.00 -> 3.05 mm
- added copper zone on In2.Cu, net +3V3
- added copper zone on B.Cu, net GND
- added copper zone on In1.Cu, net GND

Commit message: working
Parts:
- moved R33 20.2 mm to (38.0, 40.9), turned to 180 degrees
- moved R34 19.6 mm to (38.0, 42.9), turned to 180 degrees
- moved U11 12.0 mm to (41.4, 41.9), turned to 180 degrees
- moved C19 7.63 mm to (50.7, 56.8)
- moved U7 6.20 mm to (38.4, 51.2)
- moved C2 3.51 mm to (44.5, 32.2), turned to 90 degrees
- moved T3 3.14 mm to (48.0, 43.4)
- moved T1 3.13 mm to (68.9, 27.0)
- moved C10 2.67 mm to (73.6, 24.9)
- moved C9 2.62 mm to (73.6, 26.8)
- moved C8 2.61 mm to (73.6, 30.5)
- moved C7 2.60 mm to (73.6, 28.7)
- moved T2 2.58 mm to (80.7, 26.7)
- moved C22 2.54 mm to (67.8, 71.1)
- moved FB1 2.41 mm to (62.1, 29.7)
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Routing:
- net +3V3: track 0.00 -> 24.9 mm
- net GND: track 10.1 -> 27.0 mm
- net +3.3VA: track 0.00 -> 13.3 mm
- net Net-(C22-Pad1): track 0.00 -> 3.53 mm
- net Net-(C23-Pad1): track 0.00 -> 2.52 mm
- net Net-(J23-Pad1): track 0.00 -> 1.82 mm
- net Net-(J21-Pad2): track 0.00 -> 1.82 mm
