File: PCB/Waveform Generator/_autosave-Waveform Generator.kicad_pcb (KiCad board)
At the start: 4 copper layers, 80 x 104.1 mm, 141 parts, among them J1 Power input, J10 USART1_2, J12 Signal 2, J19 ADC_2, J2 RS485_1, J20 TIMER_1, J21 I2C1_1, J22 TIMER_2, J23 I2C1_2, J3 USB_B_Micro, J5 Signal 1, J6 SWD, J7 RS485_2, J8 USART1_1, J9 ADC_1, Q0 AO3401A, Q1 Q_NPN_BCE, Q2 Q_NPN_BCE, Q3 Q_PNP_BCE, Q4 Q_NPN_BCE, Q5 Q_NPN_BCE, Q6 Q_NPN_BCE, Q7 Q_NPN_BCE, Q8 Q_NPN_BCE, SW1 SW_SPDT, SW2 SW_SPDT, SW3 SW_SPDT, T0 5001, T1 5001, T2 5001, T3 5001, T4 5001, T5 5001, T6 5001, T7 5001, U1 STM32F427VITx, U10 USBLC6-2SC6, U11 USBLC6-2SC6, U2 MAX485EESAT, U3 USBLC6-2SC6, U4 OPA1602, U5 OPA1602, U6 USBLC6-2SC6, U7 USBLC6-2SC6, U8 LM335ADT, U9 USBLC6-2SC6, X1 25MHZ

Commit message: Monday morning grind
Parts:
- removed T6: 5001, Extra Components:5001 Test Point
- added ?: , , F.Cu at (-9.10, 4.50)
- added ?: , , F.Cu at (25.4, 26.9)
- added DAC_OUT_2: 5001, Extra Components:5001 Test Point, F.Cu at (72.1, 93.0)
- renumbered T2 to 3V3, T1 to 5V, T7 to DAC_OUT_1, T0 to GND, T5 to RS485_A, T4 to RS485_B, T3 to TEMP_SENSE
Other:
- board size 80 x 104.1 mm -> 80 x 105.2 mm
- board text added: "3V3"
- board text added: "5V"
- board text added: "ADC1_IN1"
- board text added: "ADC2_IN0"
- board text added: "DAC_OUT_1"
- board text added: "DAC_OUT_2"
- board text added: "GND"
- board text added: "I2C1SCL"
- board text added: "I2C1_SDA"
- board text added: "RS485_A"
- board text added: "RS485_B"
- board text added: "Waveform Generator V1 Nanodyn Systems"
- board text removed: "Waveform Generator v1 Nanodyn Systems"
Changed lines of the file:
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@@
   (general
     (thickness 1.6)
-    (drawings 9)
+    (drawings 25)
     (tracks 1100)
     (zones 0)
-    (modules 141)
+    (modules 143)
     (nets 111)
   )
@@
   (layers
     (0 F.Cu signal)
-    (1 In1.Cu power)
-    (2 In2.Cu power)
+    (1 In1.Cu power hide)
+    (2 In2.Cu power hide)
     (31 B.Cu signal)
     (32 B.Adhes user)
     (33 F.Adhes user)
-    (34 B.Paste user)
+    (34 B.Paste user hide)
     (35 F.Paste user)
     (36 B.SilkS user)
@@
   )
   (setup
-    (last_trace_width 0.3)
+    (last_trace_width 0.25)
     (user_trace_width 0.3)
     (user_trace_width 0.4)
@@
     (add_net VCC)
   )
+  (module "" (layer F.Cu)
+    (at -9.1 4.5)
+    (fp_text reference "" (at 25.4 26.9) (layer F.SilkS)
+      (effects (font (size 1.27 1.27) (thickness 0.15)))
+    )
+    (fp_text value "" (at 25.4 26.9) (layer F.SilkS)
+      (effects (font (size 1.27 1.27) (thickness 0.15)))
+    )
+  )
+  (module "" (layer F.Cu)
+    (at 25.4 26.9)
+    (fp_text reference "" (at 60.9 102.1) (layer F.SilkS)
+      (effects (font (size 1.27 1.27) (thickness 0.15)))
+    )
+    (fp_text value "" (at 60.9 102.1) (layer F.SilkS)
+      (effects (font (size 1.27 1.27) (thickness 0.15)))
+    )
+  )
   (module "Extra Components:5mm Pitch, 2 Way Terminal Block" (layer F.Cu)
     (at 60.9 102.1)
-    (fp_text reference J12 (at 0.06 -5.7) (layer F.SilkS)
+    (fp_text reference J12 (at -6.5 2.2 90) (layer F.SilkS)
       (effects (font (size 1 1) (thickness 0.15)))
     )
@@
     (tags capacitor)
     (attr smd)
-    (fp_text reference C1 (at -3.37 0.09 180) (layer F.SilkS)
+    (fp_text reference C1 (at -3 0 180) (layer F.SilkS)
       (effects (font (size 1 1) (thickness 0.15)))
     )
@@
     (tags capacitor)
     (attr smd)
-    (fp_text reference C2 (at 3.57 -0.19 180) (layer F.SilkS)
+    (fp_text reference C2 (at 3.05 0 180) (layer F.SilkS)
       (effects (font (size 1 1) (thickness 0.15)))
     )
@@
     (tags capacitor)
     (attr smd)
-    (fp_text reference C31 (at -2.35 0) (layer F.SilkS)
+    (fp_text reference C31 (at -2.4 -0.04) (layer F.SilkS)
       (effects (font (size 1 1) (thickness 0.15)))
     )
@@
   (module "Extra Components:5001 Test Point" (layer F.Cu)
     (at 36.1 94 270)
-    (fp_text reference T4 (at 3.85 0.25 180) (layer F.SilkS)
+    (fp_text reference RS485_B (at 3.5 0 180) (layer F.SilkS)
       (effects (font (size 1 1) (thickness 0.15)))
     )
@@
   (module "Extra Components:5001 Test Point" (layer F.Cu)
     (at 37.973 78.359 270)
-    (fp_text reference T5 (at 3.45 0.05 180) (layer F.SilkS)
+    (fp_text reference RS485_A (at -3.259 0.073 180) (layer F.SilkS)
       (effects (font (size 1 1) (thickness 0.15)))
     )
@@
   (module "Extra Components:5001 Test Point" (layer F.Cu)
     (at 68.9 27)
-    (fp_text reference T1 (at 0 3.65) (layer F.SilkS)
+    (fp_text reference 5V (at 0 3.65) (layer F.SilkS)
       (effects (font (size 1 1) (thickness 0.15)))
     )
@@
   (module "Extra Components:5001 Test Point" (layer F.Cu)
     (at 80.7 26.7)
-    (fp_text reference T2 (at 0 3.65) (layer F.SilkS)
+    (fp_text reference 3V3 (at 0 3.65) (layer F.SilkS)
       (effects (font (size 1 1) (thickness 0.15)))
     )
@@
   (module "Extra Components:5001 Test Point" (layer F.Cu)
     (at 48.7 42)
-    (fp_text reference T3 (at 0 3.65) (layer F.SilkS)
+    (fp_text reference TEMP_SENSE (at 0.2 4) (layer F.SilkS)
       (effects (font (size 1 1) (thickness 0.15)))
     )
@@
   (module "Extra Components:5001 Test Point" (layer F.Cu)
     (at 29.2 22.9)
-    (fp_text reference T0 (at 0.8 -3.3) (layer F.SilkS)
+    (fp_text reference GND (at 0 -3.4) (layer F.SilkS)
       (effects (font (size 1 1) (thickness 0.15)))
     )
@@
     (tags SOT-23)
     (attr smd)
-    (fp_text reference Q0 (at 2.65 0 180) (layer F.SilkS)
+    (fp_text reference Q0 (at 2.5 0.1 180) (layer F.SilkS)
       (effects (font (size 1 1) (thickness 0.15)))
     )
@@
     (tags resistor)
     (attr smd)
-    (fp_text reference R13 (at 0 1.75 180) (layer F.SilkS)
+    (fp_text reference R13 (at 0.05 1.95 180) (layer F.SilkS)
       (effects (font (size 1 1) (thickness 0.15)))
     )
@@
     (tags resistor)
     (attr smd)
-    (fp_text reference R31 (at -2.415 0) (layer F.SilkS)
+    (fp_text reference R31 (at -2.5 0) (layer F.SilkS)
       (effects (font (size 1 1) (thickness 0.15)))
     )
@@
   (module "Extra Components:TS-1109S-B-B" (layer F.Cu)
     (at 39.243 68.199 90)
-    (fp_text reference BTN0 (at -5.207 0 180) (layer F.SilkS)
+    (fp_text reference BTN0 (at 5.199 0 180) (layer F.SilkS)
       (effects (font (size 1 1) (thickness 0.15)))
     )
@@
     (tags "SOIC SO")
     (attr smd)
-    (fp_text reference U2 (at -2.686 3.816) (layer F.SilkS)
+    (fp_text reference U2 (at 0 3.35) (layer F.SilkS)
       (effects (font (size 1 1) (thickness 0.15)))
     )
@@
   (module "Extra Components:5001 Test Point" (layer F.Cu)
     (at 56.134 92.966 270)
-    (fp_text reference T7 (at 3.427 0 180) (layer F.SilkS)
-      (effects (font (size 1 1) (thickness 0.15)))
+    (fp_text reference DAC_OUT_1 (at 3.427 0 180) (layer F.SilkS)
+      (effects (font (size 0.7 0.7) (thickness 0.1)))
     )
     (fp_text value 5001 (at 0 -3.65 90) (layer F.Fab)
@@
   (module "Extra Components:5001 Test Point" (layer F.Cu)
     (at 72.136 92.964 270)
-    (fp_text reference T6 (at 3.35 0.182 180) (layer F.SilkS)
-      (effects (font (size 1 1) (thickness 0.15)))
+    (fp_text reference DAC_OUT_2 (at 3.136 -0.164 180) (layer F.SilkS)
+      (effects (font (size 0.7 0.7) (thickness 0.1)))
     )
     (fp_text value 5001 (at 0 -3.65 90) (layer F.Fab)
@@
     (tags resistor)
     (attr smd)
-    (fp_text reference R14 (at 2.4 0.05) (layer F.SilkS)
+    (fp_text reference R14 (at 2.425 -0.03) (layer F.SilkS)
       (effects (font (size 1 1) (thickness 0.15)))
     )
@@
     (tags resistor)
     (attr smd)
-    (fp_text reference R19 (at 2.35 0) (layer F.SilkS)
+    (fp_text reference R19 (at 2.445 -0.05) (layer F.SilkS)
       (effects (font (size 1 1) (thickness 0.15)))
     )
@@
     (tags resistor)
     (attr smd)
-    (fp_text reference R39 (at 3.45 0.7 180) (layer F.SilkS)
+    (fp_text reference R39 (at 3.25 0.7 180) (layer F.SilkS)
       (effects (font (size 1 1) (thickness 0.15)))
     )
@@
   (module "Extra Components:5mm Pitch, 2 Way Terminal Block" (layer F.Cu)
     (at 27.15 33.5 270)
-    (fp_text reference J23 (at -0.4 -6.9 180) (layer F.SilkS)
+    (fp_text reference J23 (at 0.2 -6.55 180) (layer F.SilkS)
       (effects (font (size 1 1) (thickness 0.15)))
     )
@@
   (module "Extra Components:5mm Pitch, 2 Way Terminal Block" (layer F.Cu)
     (at 72.410001 102.110001)
-    (fp_text reference J5 (at -2.814001 -5.844001) (layer F.SilkS)
+    (fp_text reference J5 (at 6.389999 2.789999 270) (layer F.SilkS)
       (effects (font (size 1 1) (thickness 0.15)))
     )
@@
       (net 78 "Net-(J8-Pad2)"))
   )
-  (gr_line (start 92.71 113.03) (end 17.145 113.03) (layer Edge.Cuts) (width 0.05))
+  (gr_text DAC_OUT_2 (at 75.3 113.4) (layer F.SilkS)
+    (effects (font (size 0.7 0.7) (thickness 0.12)))
+  )
+  (gr_text DAC_OUT_1 (at 63.6 113.3) (layer F.SilkS)
+    (effects (font (size 0.7 0.7) (thickness 0.12)))
+  )
+  (gr_text GND (at 69.6 113.3) (layer F.SilkS)
+    (effects (font (size 0.7 0.7) (thickness 0.12)))
+  )
+  (gr_text GND (at 58.2 113.3) (layer F.SilkS)
+    (effects (font (size 0.7 0.7) (thickness 0.12)))
+  )
+  (gr_text RS485_B (at 16.1 88.2 270) (layer F.SilkS)
+    (effects (font (size 0.7 0.7) (thickness 0.12)))
+  )
+  (gr_text RS485_A (at 16.1 82.3 270) (layer F.SilkS)
+    (effects (font (size 0.7 0.7) (thickness 0.12)))
+  )
+  (gr_text ADC1_IN1 (at 16.1 65.1 270) (layer F.SilkS)
+    (effects (font (size 0.7 0.7) (thickness 0.12)))
+  )
+  (gr_text ADC2_IN0 (at 16.1 59.2 270) (layer F.SilkS)
+    (effects (font (size 0.7 0.7) (thickness 0.12)))
+  )
+  (gr_text 5V (at 16.1 93.6 270) (layer F.SilkS)
+    (effects (font (size 0.7 0.7) (thickness 0.12)))
+  )
+  (gr_text GND (at 16.1 77 270) (layer F.SilkS)
+    (effects (font (size 0.7 0.7) (thickness 0.12)))
+  )
+  (gr_text 3V3 (at 16.1 70.3 270) (layer F.SilkS)
+    (effects (font (size 0.7 0.7) (thickness 0.12)))
+  )
+  (gr_text GND (at 16.1 53.7 270) (layer F.SilkS)
+    (effects (font (size 0.7 0.7) (thickness 0.12)))
+  )
+  (gr_text 3V3 (at 16.1 47.8 270) (layer F.SilkS)
+    (effects (font (size 0.7 0.7) (thickness 0.12)))
+  )
+  (gr_text I2C1_SDA (at 16.1 41.9 270) (layer F.SilkS)
+    (effects (font (size 0.7 0.7) (thickness 0.12)))
+  )
+  (gr_text GND (at 16 30.5 270) (layer F.SilkS)
+    (effects (font (size 0.7 0.7) (thickness 0.12)))
+  )
+  (gr_text "I2C1SCL\n" (at 16.1 36.3 270) (layer F.SilkS)
+    (effects (font (size 0.7 0.7) (thickness 0.12)))
+  )
+  (gr_line (start 92.71 114.1) (end 17.145 114.1) (layer Edge.Cuts) (width 0.05))
   (gr_line (start 95.25 10.795) (end 95.25 110.49) (layer Edge.Cuts) (width 0.05))
   (gr_line (start 17.145 8.89) (end 93.345 8.89) (layer Edge.Cuts) (width 0.05))
@@
   (gr_arc (start 17.145 111.125) (end 15.24 111.125) (angle -90) (layer Edge.Cuts) (width 0.05))
   (gr_arc (start 92.71 110.49) (end 92.71 113.03) (angle -90) (layer Edge.Cuts) (width 0.05))
-  (gr_text "Waveform Generator v1\nNanodyn Systems" (at 60.65 79.1) (layer B.SilkS)
+  (gr_text "Waveform Generator V1\nNanodyn Systems" (at 40.2 101.9) (layer B.SilkS)
     (effects (font (size 1.5 1.5) (thickness 0.3)) (justify mirror))
   )
